File: electronics/wb50.kicad_pcb (KiCad board)
At the start: 6 copper layers, 350 x 175 mm, 8 parts

Commit message: frontpanel parts placed and locked
Parts:
- added J1: IN, wb50_footprints:WB50_Jack_TRS_6pin_16.2mm, F.Cu at (36.0, 215.2)
- added J2: SW, wb50_footprints:WB50_Jack_TRS_6pin_16.2mm, F.Cu at (66.0, 215.2)
- moved RV1 363.0 mm to (396.0, 219.7)
- moved RV2 275.9 mm to (356.0, 219.7)
- moved RV8 247.0 mm to (116.0, 219.7)
- moved RV3 188.7 mm to (316.0, 219.7)
- moved RV7 159.9 mm to (156.0, 219.7)
- moved RV4 101.6 mm to (276.0, 219.7)
- moved RV6 72.7 mm to (196.0, 219.7)
- moved RV5 14.4 mm to (236.0, 219.7)
Other:
- board size 350 x 175 mm -> 380 x 175 mm

Commit message: bring potentiometers more to front and lock again
Parts:
- moved RV1 1.35 mm to (396.0, 221.0)
- moved RV2 1.35 mm to (356.0, 221.0)
- moved RV3 1.35 mm to (316.0, 221.0)
- moved RV4 1.35 mm to (276.0, 221.0)
- moved RV5 1.35 mm to (236.0, 221.0)
- moved RV6 1.35 mm to (196.0, 221.0)
- moved RV7 1.35 mm to (156.0, 221.0)
- moved RV8 1.35 mm to (116.0, 221.0)
Changed lines of the file:
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@@
 		(allow_soldermask_bridges_in_footprints no)
 		(tenting front back)
-		(grid_origin 66 216.6)
+		(grid_origin 24.6 226)
 		(pcbplotparams
 			(layerselection 0x00000000_00000000_55555555_5755f5ff)
@@
 		(locked yes)
 		(layer "F.Cu")
-		(at 276 219.65)
+		(at 276 221)
 		(property "Reference" "RV4"
 			(at 0 -6.8 0)
@@
 		(locked yes)
 		(layer "F.Cu")
-		(at 396 219.65)
+		(at 396 221)
 		(property "Reference" "RV1"
 			(at 0 -6.8 0)
@@
 		(locked yes)
 		(layer "F.Cu")
-		(at 316 219.65)
+		(at 316 221)
 		(property "Reference" "RV3"
 			(at 0 -6.8 0)
@@
 		(locked yes)
 		(layer "F.Cu")
-		(at 356 219.65)
+		(at 356 221)
 		(property "Reference" "RV2"
 			(at 0 -6.8 0)
@@
 		(locked yes)
 		(layer "F.Cu")
-		(at 156 219.65)
+		(at 156 221)
 		(property "Reference" "RV7"
 			(at 0 -6.8 0)
@@
 		(locked yes)
 		(layer "F.Cu")
-		(at 236 219.65)
+		(at 236 221)
 		(property "Reference" "RV5"
 			(at 0 -6.8 0)
@@
 		(locked yes)
 		(layer "F.Cu")
-		(at 196 219.65)
+		(at 196 221)
 		(property "Reference" "RV6"
 			(at 0 -6.8 0)
@@
 		(locked yes)
 		(layer "F.Cu")
-		(at 116 219.65)
+		(at 116 221)
 		(property "Reference" "RV8"
 			(at 0 -6.8 0)

Commit message: adjust pcb size
Parts:
- moved J1 4.77 mm to (31.4, 214.0)
- moved J2 4.77 mm to (61.4, 214.0)
- moved RV1 4.60 mm to (391.4, 221.0)
- moved RV2 4.60 mm to (351.4, 221.0)
- moved RV3 4.60 mm to (311.4, 221.0)
- moved RV4 4.60 mm to (271.4, 221.0)
- moved RV5 4.60 mm to (231.4, 221.0)
- moved RV6 4.60 mm to (191.4, 221.0)
- moved RV7 4.60 mm to (151.4, 221.0)
- moved RV8 4.60 mm to (111.4, 221.0)
Other:
- board size 380 x 175 mm -> 394 x 100 mm
Changed lines of the file:
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@@
 		(allow_soldermask_bridges_in_footprints no)
 		(tenting front back)
-		(grid_origin 24.6 226)
+		(grid_origin 13 226)
 		(pcbplotparams
 			(layerselection 0x00000000_00000000_55555555_5755f5ff)
@@
 		(locked yes)
 		(layer "F.Cu")
-		(at 36 215.25)
+		(at 31.4 214)
 		(property "Reference" "J1"
 			(at -0.8 0 0)
@@
 		(locked yes)
 		(layer "F.Cu")
-		(at 276 221)
+		(at 271.4 221)
 		(property "Reference" "RV4"
 			(at 0 -6.8 0)
@@
 		(locked yes)
 		(layer "F.Cu")
-		(at 396 221)
+		(at 391.4 221)
 		(property "Reference" "RV1"
 			(at 0 -6.8 0)
@@
 		(locked yes)
 		(layer "F.Cu")
-		(at 316 221)
+		(at 311.4 221)
 		(property "Reference" "RV3"
 			(at 0 -6.8 0)
@@
 		(locked yes)
 		(layer "F.Cu")
-		(at 356 221)
+		(at 351.4 221)
 		(property "Reference" "RV2"
 			(at 0 -6.8 0)
@@
 		(locked yes)
 		(layer "F.Cu")
-		(at 156 221)
+		(at 151.4 221)
 		(property "Reference" "RV7"
 			(at 0 -6.8 0)
@@
 		(locked yes)
 		(layer "F.Cu")
-		(at 66 215.25)
+		(at 61.4 214)
 		(property "Reference" "J2"
 			(at -0.8 0 0)
@@
 		(locked yes)
 		(layer "F.Cu")
-		(at 236 221)
+		(at 231.4 221)
 		(property "Reference" "RV5"
 			(at 0 -6.8 0)
@@
 		(locked yes)
 		(layer "F.Cu")
-		(at 196 221)
+		(at 191.4 221)
 		(property "Reference" "RV6"
 			(at 0 -6.8 0)
@@
 		(locked yes)
 		(layer "F.Cu")
-		(at 116 221)
+		(at 111.4 221)
 		(property "Reference" "RV8"
 			(at 0 -6.8 0)
@@
 	)
 	(gr_rect
-		(start 24.6 51)
-		(end 404.6 226)
+		(start 13 126)
+		(end 407 226)
 		(stroke
 			(width 0.2)

Commit message: updated pcb size
Parts:
- moved J1 121.9 mm to (142.9, 263.2)
- moved J2 121.9 mm to (172.9, 263.2)
- moved RV1 121.9 mm to (502.9, 270.2)
- moved RV2 121.9 mm to (462.9, 270.2)
- moved RV3 121.9 mm to (422.9, 270.2)
- moved RV4 121.9 mm to (382.9, 270.2)
- moved RV8 121.9 mm to (222.9, 270.2)
- moved RV5 121.9 mm to (342.9, 270.2)
- moved RV6 121.9 mm to (302.9, 270.2)
- moved RV7 121.9 mm to (262.9, 270.2)
Other:
- board size 394 x 100 mm -> 405 x 100 mm
Changed lines of the file:
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@@
 		(legacy_teardrops no)
 	)
-	(paper "A3")
+	(paper "A2")
 	(layers
 		(0 "F.Cu" signal)
@@
 		(locked yes)
 		(layer "F.Cu")
-		(at 31.4 214)
+		(at 142.9 263.2)
 		(property "Reference" "J1"
 			(at -0.8 0 0)
@@
 		(locked yes)
 		(layer "F.Cu")
-		(at 271.4 221)
+		(at 382.9 270.2)
 		(property "Reference" "RV4"
 			(at 0 -6.8 0)
@@
 		(locked yes)
 		(layer "F.Cu")
-		(at 391.4 221)
+		(at 502.9 270.2)
 		(property "Reference" "RV1"
 			(at 0 -6.8 0)
@@
 		(locked yes)
 		(layer "F.Cu")
-		(at 311.4 221)
+		(at 422.9 270.2)
 		(property "Reference" "RV3"
 			(at 0 -6.8 0)
@@
 		(locked yes)
 		(layer "F.Cu")
-		(at 351.4 221)
+		(at 462.9 270.2)
 		(property "Reference" "RV2"
 			(at 0 -6.8 0)
@@
 		(locked yes)
 		(layer "F.Cu")
-		(at 151.4 221)
+		(at 262.9 270.2)
 		(property "Reference" "RV7"
 			(at 0 -6.8 0)
@@
 		(locked yes)
 		(layer "F.Cu")
-		(at 61.4 214)
+		(at 172.9 263.2)
 		(property "Reference" "J2"
 			(at -0.8 0 0)
@@
 		(locked yes)
 		(layer "F.Cu")
-		(at 231.4 221)
+		(at 342.9 270.2)
 		(property "Reference" "RV5"
 			(at 0 -6.8 0)
@@
 		(locked yes)
 		(layer "F.Cu")
-		(at 191.4 221)
+		(at 302.9 270.2)
 		(property "Reference" "RV6"
 			(at 0 -6.8 0)
@@
 		(locked yes)
 		(layer "F.Cu")
-		(at 111.4 221)
+		(at 222.9 270.2)
 		(property "Reference" "RV8"
 			(at 0 -6.8 0)
@@
 	)
 	(gr_rect
-		(start 13 126)
-		(end 407 226)
+		(start 119.5 176)
+		(end 524.5 276)
 		(stroke
 			(width 0.2)
@@
 		)
 		(fill no)
+		(locked yes)
 		(layer "Edge.Cuts")
 	)
