File: electronics/backpanel/wb50_back.kicad_sch (KiCad schematic)
At the start: 0 parts

Commit message: routed
Parts:
- added J1, J2: Audio Jack TRS, 6pin (with switches), wb50_footprints:WB50_Jack_TRS_6pin_16.2mm, symbol wb50_symbols:WB50_Jack_TRS_6pin_Switched
- added X1: Audio IN, TestPoint:TestPoint_THTPad_D4.0mm_Drill2.0mm, symbol Connector:TestPoint
- added X2: GND_OT, TestPoint:TestPoint_THTPad_D4.0mm_Drill2.0mm, symbol Connector:TestPoint
- added X3: NFB, TestPoint:TestPoint_THTPad_D1.5mm_Drill0.7mm, symbol Connector:TestPoint
- added X4: GND_NFB, TestPoint:TestPoint_THTPad_D4.0mm_Drill2.0mm, symbol Connector:TestPoint
Connections:
- new net: J1.1, J2.1, J2.6, X2.1, X4.1
- new net: J1.2, J1.3, J1.4, J1.5, J2.2, J2.3, X1.1, X3.1
- new net: J1.6, J2.4, J2.5
Other:
- note added: "GND vom OT Sternpunkt"
- note added: "Kabel von Impedanzwahlschalter"
- note added: "NFB hier NUR Seele verbinden. NFB Schirm wird nur auf der Hauptplatine verbunden. Externes GND Kabel parallel zu NFB führen für mögliche Ströme."
