File: electronics/backpanel/wb50_back.kicad_pcb (KiCad board)
At the start: 2 copper layers, 56.5 x 34.2 mm, 6 parts, among them J1 Audio Jack TRS, 6pin (with sw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, J2 Audio Jack TRS, 6pin (with sw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, X1 Audio IN, X2 GND_OT, X3 NFB, X4 GND_NFB

Commit message: setup jlcpcb
Other:
- board text added: "C.Müller 2025"
- board text added: "WB50-Speaker Connector V1.0"
Changed lines of the file:
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@@
 		(layer "Edge.Cuts")
+	)
+	(gr_text "C.Müller 2025"
+		(at 125.25 137.25 90)
+		(layer "F.SilkS")
+		(effects
+			(font
+				(size 1 1)
+				(thickness 0.2)
+				(bold yes)
+			)
+			(justify left bottom)
+		)
+	)
+	(gr_text "WB50-Speaker Connector V1.0"
+		(at 102.5 128.75 90)
+		(layer "F.SilkS")
+		(effects
+			(font
+				(size 1 1)
+				(thickness 0.2)
+			)
+			(justify left bottom)
+		)
 	)
 	(segment
