File: electronics/main/schematics/controls.kicad_sch (KiCad schematic)
At the start: 8 parts

Commit message: PI stage ready
Parts:
- removed RV1: Presence, wb50_footprints:WB50_Pot_Omeg_PC20BU_P5.00mm, symbol Device:R_Potentiometer
- removed RV2: Bass, wb50_footprints:WB50_Pot_Omeg_PC20BU_P5.00mm, symbol Device:R_Potentiometer
- removed RV3: Mid, wb50_footprints:WB50_Pot_Omeg_PC20BU_P5.00mm, symbol Device:R_Potentiometer
- removed RV4: Treble, wb50_footprints:WB50_Pot_Omeg_PC20BU_P5.00mm, symbol Device:R_Potentiometer
- removed RV5: Vol1, wb50_footprints:WB50_Pot_Omeg_PC20BU_P5.00mm, symbol Device:R_Potentiometer
- removed RV6: Vol2, wb50_footprints:WB50_Pot_Omeg_PC20BU_P5.00mm, symbol Device:R_Potentiometer
- removed RV7: Gain1, wb50_footprints:WB50_Pot_Omeg_PC20BU_P5.00mm, symbol Device:R_Potentiometer
- removed RV8: Gain2, wb50_footprints:WB50_Pot_Omeg_PC20BU_P5.00mm, symbol Device:R_Potentiometer
