File: electronics/main/schematics/powerAmp.kicad_sch (KiCad schematic)
At the start: 2 parts

Commit message: schematic ready? - check
Parts:
- added Audio-A, Audio-B: 1, TestPoint:TestPoint_THTPad_D3.0mm_Drill1.5mm, symbol Connector:TestPoint_Small
- added BiasA, BiasB, GND-Mess: 1, TestPoint:TestPoint_Pad_D2.0mm, symbol Connector:TestPoint_Small
- added R22, R23: CFR-25JT-52-1K5, footprints:RES-TH_BD2.4-L6.3-P10.30-D0.6, symbol jlcpcb:CFR-25JT-52-1K5
- added R30, R31: MF1/4W-1Ω±1%-ST26, footprints:RES-TH_BD2.7-L6.2-P10.20-D0.4, symbol jlcpcb:MF1/4W-1Ω±1%-ST26
- added U27, U28: CR1/2W-220K±5%-XT52, footprints:RES-TH_BD3.5-L9.0-P13.00-D0.5, symbol jlcpcb:CR1/2W-220K±5%-XT52
- added U29, U30: CR-L5W-1KΩJ, footprints:RES-TH_BD9.5-L22.0-P26.00-D0.7, symbol jlcpcb:CR-L5W-1KΩJ
Connections:
- net HEAT1: now reaches V4.2 (f)
- net HEAT1: now also V5.2 (f)
- net HEAT2: now reaches V4.7 (f)
- net HEAT2: now also V5.7 (f)
- net at V5.1 (g3): now also V5.8 (k), BiasB.1, R31.2
- net at V5.3 (a): now also Audio-B.1
- net at V5.4 (g2): now also U30.2
- net at V5.5 (g1): now also R23.2
- net at V4.1 (g3): now also V4.8 (k), BiasA.1, R30.1
- net at V4.3 (a): now also Audio-A.1
- net at V4.4 (g2): now also U29.1
- net at V4.5 (g1): now also R22.2
- new net A_IN: R22.1, U27.1
- new net B_IN: R23.1, U28.2
- new net Bias-Set: U27.2, U28.1
- new net GND-AUD: GND-Mess.1, R30.2, R31.1
- new net HV-B: U29.2, U30.1
Other:
- moved on the sheet: V4A, V4B, V5A, V5B

Commit message: schematic  checked!
Parts:
- added HV-OT1, HV-OT2: 1, TestPoint:TestPoint_THTPad_D3.0mm_Drill1.5mm, symbol Connector:TestPoint_Small
- renumbered Audio-A to Audio-A1, Audio-B to Audio-B1, BiasA to BiasA1, BiasB to BiasB1, GND-Mess to GND-Mess1
Connections:
- new net HV-A: HV-OT1.1, HV-OT2.1
Other:
- moved on the sheet: Audio-A1, Audio-B1, BiasA1, BiasB1, GND-Mess1, R22, R23, R30, R31, U27, U28, U29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
