File: electronics/main/schematics/phaseInverter.kicad_sch (KiCad schematic)
At the start: 1 part

Commit message: PI stage ready
Parts:
- added R16: CR1W-10M±5%-6T63, footprints:RES-TH_BD4.5-L11.0-P15.00-D0.7, symbol jlcpcb:CR1W-10M±5%-6T63
- added R17, R18: 1Meg 500V 250mW, footprints:RES-TH_BD2.4-L6.3-P10.30-D0.6, symbol jlcpcb:CFR-25JT-52-1M
- added R19: CF3WS-10KΩ±5%_T, footprints:RES-TH_BD5.5-L15.0-P19.00-D0.8, symbol jlcpcb:CF3WS-10KΩ±5%_T
- added R20: CR1W-100K±5%-TT63, footprints:RES-TH_BD4.5-L11.0-P15.00-D0.7, symbol jlcpcb:CR1W-100K±5%-TT63
- added R21: CR1/4W-47K±5%-ST52, footprints:RES-TH_BD2.7-L6.2-P10.20-D0.4, symbol jlcpcb:CR1/4W-47K±5%-ST52
- added RV1: Presence, wb50_footprints:WB50_Pot_Omeg_PC20BU_P5.00mm, symbol Device:R_Potentiometer
- added U17, U25, U26: 22n 630V 5%, wb50_footprints:MUSTARD_CAP_D8.5_L20.5_P25.5, symbol wb50_symbols:YellowCap_4n7_630V
- added U18: 470R 500V 2W, footprints:RES-TH_BD5.0-L15.5-P19.50-D0.7, symbol jlcpcb:CFR02SJ0471A10
- added U19, U23: 100n 630V 5%, wb50_footprints:MUSTARD_CAP_D10_L32_P40.4, symbol wb50_symbols:YellowCap_100n_630V
- added U20: CF2WS-82KΩ±5%_T, footprints:RES-TH_BD4.0-L11.5-P15.50-D0.7, symbol jlcpcb:CF2WS-82KΩ±5%_T
- added U21: 100pF 500V 5%, wb50_footprints:MICA_CAP_L15.5_W3.6_P8.7, symbol wb50_symbols:MicaCap_500pf_500V
- added U22: CR1/2W-220K±5%-XT52, footprints:RES-TH_BD3.5-L9.0-P13.00-D0.5, symbol jlcpcb:CR1/2W-220K±5%-XT52
- added U24: 4n7 630V 5%, wb50_footprints:MUSTARD_CAP_D8.5_L20.5_P25.5, symbol wb50_symbols:YellowCap_4n7_630V
Connections:
- net +12V: now reaches V3.4 (H1)
- net GND-AUX: now reaches V3.5 (H2)
- net at V3.1 (A/P): now also U20.2, U21.1
- net at V3.2 (G): now also R17.1, U17.2
- net at V3.3 (C/K): now also V3.8 (C/K), U18.1
- net at V3.6 (A/P): now also R20.2, U21.2, U26.1
- net at V3.7 (G): now also R18.1, U23.1
- new net: R21.2, U22.1, U24.1
- new net: R19.2, R21.1, RV1.1, U23.2
- new net: RV1.2, U19.1
- new net: R17.2, R18.2, R19.1, U18.2
- new net GND-AUD: R16.2, RV1.3, U19.2
- new net HV-C: R20.1, U20.1, U25.1
- new net NFB_OUT: U22.2, U24.2
- new net PI_IN: R16.1, U17.1
- new net PI_OUT_A: U25.2
- new net PI_OUT_B: U26.2
Other:
- moved on the sheet: V3A, V3B, V3C

Commit message: schematic  checked!
Parts:
- added THUMP1, THUMP2: 1, TestPoint:TestPoint_THTPad_D2.0mm_Drill1.0mm, symbol Connector:TestPoint_Small
Connections:
- net HV-C: no longer U25.1
- net NFB_OUT: now also THUMP2.1
- net at R21.2, U22.1, U24.1: now also THUMP1.1
- net at U20.2, U21.1, V3.1 (A/P): now also U25.1
Other:
- moved on the sheet: U20
Changed lines of the file:
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@@
-	)
-	(junction
-		(at 124.46 55.88)
-		(diameter 0)
-		(color 0 0 0 0)
-	)
-	(junction
-		(at 114.3 53.34)
-		(diameter 0)
-		(color 0 0 0 0)
 	)
 	(junction
@@
 	)
 	(junction
+		(at 114.3 41.91)
+		(diameter 0)
+		(color 0 0 0 0)
+	)
+	(junction
+		(at 104.14 55.88)
+		(diameter 0)
+		(color 0 0 0 0)
+	)
+	(junction
 		(at 124.46 73.66)
 		(diameter 0)
@@
 	(wire
 		(pts
+			(xy 104.14 55.88) (xy 158.75 55.88)
+		)
+		(stroke
+			(width 0)
+			(type default)
+		)
+	)
+	(wire
+		(pts
 			(xy 114.3 95.25) (xy 114.3 99.06)
 		)
@@
 	(wire
 		(pts
-			(xy 104.14 53.34) (xy 114.3 53.34)
+			(xy 104.14 41.91) (xy 114.3 41.91)
 		)
 		(stroke
@@
 	(wire
 		(pts
-			(xy 114.3 53.34) (xy 114.3 43.18)
-		)
-		(stroke
-			(width 0)
-			(type default)
-		)
-	)
-	(wire
-		(pts
 			(xy 168.91 55.88) (xy 231.14 55.88)
 		)
@@
 	(wire
 		(pts
+			(xy 199.39 114.3) (xy 199.39 127)
+		)
+		(stroke
+			(width 0)
+			(type default)
+		)
+	)
+	(wire
+		(pts
 			(xy 219.71 127) (xy 229.87 127)
 		)
@@
 	(wire
 		(pts
-			(xy 124.46 57.15) (xy 124.46 55.88)
-		)
-		(stroke
-			(width 0)
-			(type default)
-		)
-	)
-	(wire
-		(pts
-			(xy 104.14 67.31) (xy 104.14 73.66)
+			(xy 124.46 41.91) (xy 124.46 57.15)
+		)
+		(stroke
+			(width 0)
+			(type default)
+		)
+	)
+	(wire
+		(pts
+			(xy 104.14 53.34) (xy 104.14 55.88)
 		)
 		(stroke
@@
 	(wire
 		(pts
-			(xy 104.14 57.15) (xy 104.14 53.34)
+			(xy 104.14 43.18) (xy 104.14 41.91)
 		)
 		(stroke
@@
 	(wire
 		(pts
-			(xy 124.46 53.34) (xy 114.3 53.34)
-		)
-		(stroke
-			(width 0)
-			(type default)
-		)
-	)
-	(wire
-		(pts
-			(xy 124.46 55.88) (xy 158.75 55.88)
-		)
-		(stroke
-			(width 0)
-			(type default)
-		)
-	)
-	(wire
-		(pts
-			(xy 124.46 55.88) (xy 124.46 53.34)
+			(xy 124.46 41.91) (xy 114.3 41.91)
+		)
+		(stroke
+			(width 0)
+			(type default)
+		)
+	)
+	(wire
+		(pts
+			(xy 114.3 41.91) (xy 114.3 25.4)
 		)
 		(stroke
@@
 	(wire
 		(pts
+			(xy 229.87 114.3) (xy 229.87 127)
+		)
+		(stroke
+			(width 0)
+			(type default)
+		)
+	)
+	(wire
+		(pts
 			(xy 114.3 109.22) (xy 114.3 111.76)
 		)
@@
 		(pts
 			(xy 104.14 73.66) (xy 109.22 73.66)
+		)
+		(stroke
+			(width 0)
+			(type default)
+		)
+	)
+	(wire
+		(pts
+			(xy 104.14 55.88) (xy 104.14 73.66)
 		)
 		(stroke
@@
 	(global_label "HV-C"
 		(shape passive)
-		(at 114.3 43.18 90)
+		(at 114.3 25.4 90)
 		(fields_autoplaced yes)
 		(effects
@@
 		)
 		(property "Intersheetrefs" "${INTERSHEET_REFS}"
-			(at 114.3 36.0446 90)
+			(at 114.3 18.2646 90)
 			(effects
 				(font
@@
 	)
 	(symbol
+		(lib_id "Connector:TestPoint_Small")
+		(at 199.39 114.3 90)
+		(unit 1)
+		(exclude_from_sim no)
+		(in_bom yes)
+		(on_board yes)
+		(dnp no)
+		(fields_autoplaced yes)
+		(property "Reference" "THUMP1"
+			(at 199.39 109.22 90)
+			(effects
+				(font
+					(size 1.27 1.27)
+				)
+			)
+		)
+		(property "Value" "1"
+			(at 199.39 111.76 90)
+			(effects
+				(font
+					(size 1.27 1.27)
+				)
+			)
+		)
+		(property "Footprint" "TestPoint:TestPoint_THTPad_D2.0mm_Drill1.0mm"
+			(at 199.39 109.22 0)
+			(effects
+				(font
+					(size 1.27 1.27)
+				)
+				(hide yes)
+			)
+		)
+		(property "Datasheet" "~"
+			(at 199.39 109.22 0)
+			(effects
+				(font
+					(size 1.27 1.27)
+				)
+				(hide yes)
+			)
+		)
+		(property "Description" "test point"
+			(at 199.39 114.3 0)
+			(effects
+				(font
+					(size 1.27 1.27)
+				)
+				(hide yes)
+			)
+		)
+		(pin "1"
+		)
+		(instances
+			(project "wb50"
+				(path "/6805e3ef-87bd-473d-890f-05ae2da73c1a/94f97982-768b-42a9-8fe1-8b9d029f0dfa"
+					(reference "THUMP1")
+					(unit 1)
+				)
+			)
+		)
+	)
+	(symbol
+		(lib_id "Connector:TestPoint_Small")
+		(at 229.87 114.3 90)
+		(unit 1)
+		(exclude_from_sim no)
+		(in_bom yes)
+		(on_board yes)
+		(dnp no)
+		(fields_autoplaced yes)
+		(property "Reference" "THUMP2"
+			(at 229.87 109.22 90)
+			(effects
+				(font
+					(size 1.27 1.27)
+				)
+			)
+		)
+		(property "Value" "1"
+			(at 229.87 111.76 90)
+			(effects
+				(font
+					(size 1.27 1.27)
+				)
+			)
+		)
+		(property "Footprint" "TestPoint:TestPoint_THTPad_D2.0mm_Drill1.0mm"
+			(at 229.87 109.22 0)
+			(effects
+				(font
+					(size 1.27 1.27)
+				)
+				(hide yes)
+			)
+		)
+		(property "Datasheet" "~"
+			(at 229.87 109.22 0)
+			(effects
+				(font
+					(size 1.27 1.27)
+				)
+				(hide yes)
+			)
+		)
+		(property "Description" "test point"
+			(at 229.87 114.3 0)
+			(effects
+				(font
+					(size 1.27 1.27)
+				)
+				(hide yes)
+			)
+		)
+		(pin "1"
+		)
+		(instances
+			(project "wb50"
+				(path "/6805e3ef-87bd-473d-890f-05ae2da73c1a/94f97982-768b-42a9-8fe1-8b9d029f0dfa"
+					(reference "THUMP2")
+					(unit 1)
+				)
+			)
+		)
+	)
+	(symbol
 		(lib_id "jlcpcb:CF2WS-82KΩ±5%_T")
-		(at 104.14 62.23 270)
+		(at 104.14 48.26 270)
 		(unit 1)
 		(exclude_from_sim no)
@@
 		(dnp no)
 		(property "Reference" "U20"
-			(at 97.282 60.96 90)
+			(at 97.282 46.99 90)
 			(effects
 				(font
@@
 		)
 		(property "Value" "CF2WS-82KΩ±5%_T"
-			(at 81.534 63.5 90)
+			(at 81.534 49.53 90)
 			(effects
 				(font
@@
 		)
 		(property "Footprint" "footprints:RES-TH_BD4.0-L11.5-P15.50-D0.7"
-			(at 93.98 62.23 0)
+			(at 93.98 48.26 0)
 			(effects
 				(font
@@
 		)
 		(property "Datasheet" "https://item.szlcsc.com/59784.html"
-			(at 104.267 59.944 0)
+			(at 104.267 45.974 0)
 			(effects
 				(font
@@
 		)
 		(property "Description" ""
-			(at 104.14 62.23 0)
+			(at 104.14 48.26 0)
 			(effects
 				(font
@@
 		)
 		(property "LCSC" "C120647"
-			(at 104.14 62.23 0)
-			(effects
-				(font
+			(at 104.14 48.26 0)
+			(effects
+				(font

Commit message: updated PCB
Parts:
- THUMP1, THUMP2: footprint TestPoint:TestPoint_THTPad_D2.0mm_Drill1.0mm -> TestPoint:TestPoint_THTPad_D3.0mm_Drill1.5mm
Changed lines of the file:
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@@
 			)
 		)
-		(property "Footprint" "TestPoint:TestPoint_THTPad_D2.0mm_Drill1.0mm"
+		(property "Footprint" "TestPoint:TestPoint_THTPad_D3.0mm_Drill1.5mm"
 			(at 199.39 109.22 0)
 			(effects
@@
 			)
 		)
-		(property "Footprint" "TestPoint:TestPoint_THTPad_D2.0mm_Drill1.0mm"
+		(property "Footprint" "TestPoint:TestPoint_THTPad_D3.0mm_Drill1.5mm"
 			(at 229.87 109.22 0)
 			(effects
