File: electronics/main/schematics/preamp.kicad_sch (KiCad schematic)
At the start: 2 parts

Commit message: widerstände angelegt
Connections:
- net +12V: now reaches V1.4 (H1)
- net +12V: now also V2.4 (H1)
- net GND-AUX: now reaches V1.5 (H2)
- net GND-AUX: now also V2.5 (H2)
Other:
- moved on the sheet: V1C

Commit message: PI stage ready
Parts:
- removed V2: 12AX7, wb50_footprints:WB50_Socket_Noval_9Pin_D21.0mm_Hole1.8mm, symbol wb50_symbols:WB50_12AX7
- added C5, C6: 0,82uF 400V 20 %, footprints:CAP-TH_BD6.3-P2.50-D1.0-FD, symbol jlcpcb:10uf/100V
- added R1, R6: 33k 500V 2W, footprints:RES-TH_BD3.0-L9.5-P13.50-D0.6, symbol jlcpcb:CFR02SJ0333A10
- added R2: 1Meg 500V 250mW, footprints:RES-TH_BD2.4-L6.3-P10.30-D0.6, symbol jlcpcb:CFR-25JT-52-1M
- added R3, R5, R9: CR1W-100K±5%-TT63, footprints:RES-TH_BD4.5-L11.0-P15.00-D0.7, symbol jlcpcb:CR1W-100K±5%-TT63
- added R4, R8: CR1/4W-2K7±5%-ST26, footprints:RES-TH_BD2.7-L6.2-P10.20-D0.4, symbol jlcpcb:CR1/4W-2K7±5%-ST26
- added R7: CR1W-10M±5%-6T63, footprints:RES-TH_BD4.5-L11.0-P15.00-D0.7, symbol jlcpcb:CR1W-10M±5%-6T63
- added RELAY1, RELAY2: G5V-1-12V, footprints:RELAY-TH_G5V-1, symbol jlcpcb:G5V-1-12V
- added RV7: Gain1, wb50_footprints:WB50_Pot_Omeg_PC20BU_P5.00mm, symbol Device:R_Potentiometer
- added RV8: Gain2, wb50_footprints:WB50_Pot_Omeg_PC20BU_P5.00mm, symbol Device:R_Potentiometer
- added U10: 250pF 500V 5%, wb50_footprints:MICA_CAP_L15.5_W3.6_P8.7, symbol wb50_symbols:MicaCap_500pf_500V
- added U4: CR1/2W-220K±5%-XT52, footprints:RES-TH_BD3.5-L9.0-P13.00-D0.5, symbol jlcpcb:CR1/2W-220K±5%-XT52
- added U5: CR2W-68K±5%-9T73, footprints:RES-TH_BD5.0-L15.5-P19.50-D0.7, symbol jlcpcb:CR2W-68K±5%-9T73
- added U6, U9: 500pF 500V 5%, wb50_footprints:MICA_CAP_L15.5_W3.6_P8.7, symbol wb50_symbols:MicaCap_500pf_500V
- added U7: 4n7 630V 5%, wb50_footprints:MUSTARD_CAP_D8.5_L20.5_P25.5, symbol wb50_symbols:YellowCap_4n7_630V
- added U8: 2n2 630V 5%, wb50_footprints:MUSTARD_CAP_D8.5_L20.5_P25.5, symbol wb50_symbols:YellowCap_4n7_630V
- added X-BS-1: 1, symbol Connector:TestPoint_Small
- added X-BS-2: 2, symbol Connector:TestPoint_Small
- added X-BS-3: 3, symbol Connector:TestPoint_Small
Connections:
- net Audio_IN: now also R1.1, R2.1, RELAY1.10
- net GND-AUD: now also C5.2, C6.2, R2.2, R4.2, R7.2, R8.2, RV7.1, RV8.1
- net at V1.6 (A/P): now also R9.2, U8.1
- net at V1.7 (G): now also R6.2
- net at V1.8 (C/K): now also C6.1, R8.1
- net at V1.1 (A/P): now also R3.2, U6.2, U7.1
- net at V1.2 (G): now also R1.2
- net at V1.3 (C/K): now also C5.1, R4.1
- new net: R5.2, RELAY1.1
- new net: R6.1, R7.1, RELAY1.5, RELAY1.6
- new net: R3.1, U4.2, U6.1
- new net: U5.1, U7.2
- new net: R5.1, U5.2
- new net: U9.2, X-BS-3.1
- new net: RV7.3, RV8.3, U10.1, U8.2, U9.1
- new net: U10.2, X-BS-1.1
- new net: RELAY2.10, RV7.2, X-BS-2.1
- new net: RELAY2.1, RV8.2
- new net HV-E: R9.1, U4.1
- new net PreAmp_OUT: RELAY2.5, RELAY2.6
Other:
- note added: "Bright Switch Solder Points"
- moved on the sheet: V1A, V1B, V1C

Commit message: schematic ready? - check
Parts:
- X-BS-1, X-BS-2, X-BS-3: footprint (none) -> TestPoint:TestPoint_THTPad_D2.0mm_Drill1.0mm
Changed lines of the file:
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@@
 			)
 		)
-		(property "Footprint" ""
+		(property "Footprint" "TestPoint:TestPoint_THTPad_D2.0mm_Drill1.0mm"
 			(at 302.26 140.97 0)
 			(effects
@@
 			)
 		)
-		(property "Footprint" ""
+		(property "Footprint" "TestPoint:TestPoint_THTPad_D2.0mm_Drill1.0mm"
 			(at 313.69 143.51 0)
 			(effects
@@
 			)
 		)
-		(property "Footprint" ""
+		(property "Footprint" "TestPoint:TestPoint_THTPad_D2.0mm_Drill1.0mm"
 			(at 302.26 147.32 0)
 			(effects

Commit message: schematic  checked!
Parts:
- added D4, D5: UF4007_C960666, footprints:DO-41_BD2.4-L4.7-P8.70-D0.9-RD, symbol jlcpcb:UF4007_C960666
Connections:
- net +12V: now also RELAY1.2, RELAY2.2, D4.1 (K), D5.1 (K)
- net GND-AUD: now also R5.2
- net at RELAY1.1: now also R5.1, U5.2; no longer R5.2
- net REL-SW: now reaches RELAY1.9
- net REL-SW: now also RELAY2.9, D4.2 (A), D5.2 (A)
Other:
- moved on the sheet: R5, R7

Commit message: updated PCB
Parts:
- added N2: ~, wb50_footprints:NetTie_0.5mm_2Pad, symbol wb50_symbols:NetTie
- X-BS-1, X-BS-2, X-BS-3: footprint TestPoint:TestPoint_THTPad_D2.0mm_Drill1.0mm -> TestPoint:TestPoint_THTPad_D3.0mm_Drill1.5mm
Connections:
- net GND-AUD: now also N2.2 (Net2)
- new net GND-PWR: N2.1 (Net1)
Changed lines of the file:
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@@
 	(wire
 		(pts
+			(xy 62.23 53.34) (xy 59.69 53.34)
+		)
+		(stroke
+			(width 0)
+			(type default)
+		)
+	)
+	(wire
+		(pts
 			(xy 156.21 104.14) (xy 156.21 96.52)
 		)
@@
 	(wire
 		(pts
+			(xy 72.39 53.34) (xy 67.31 53.34)
+		)
+		(stroke
+			(width 0)
+			(type default)
+		)
+	)
+	(wire
+		(pts
 			(xy 74.93 130.81) (xy 74.93 133.35)
 		)
@@
 	(wire
 		(pts
+			(xy 72.39 55.88) (xy 72.39 53.34)
+		)
+		(stroke
+			(width 0)
+			(type default)
+		)
+	)
+	(wire
+		(pts
 			(xy 156.21 96.52) (xy 179.07 96.52)
 		)
@@
 	(wire
 		(pts
+			(xy 59.69 53.34) (xy 59.69 55.88)
+		)
+		(stroke
+			(width 0)
+			(type default)
+		)
+	)
+	(wire
+		(pts
 			(xy 330.2 134.62) (xy 330.2 139.7)
 		)
@@
 	)
 	(symbol
+		(lib_id "power:GND")
+		(at 59.69 55.88 0)
+		(unit 1)
+		(exclude_from_sim no)
+		(in_bom yes)
+		(on_board yes)
+		(dnp no)
+		(property "Reference" "#PWR047"
+			(at 59.69 62.23 0)
+			(effects
+				(font
+					(size 1.27 1.27)
+				)
+				(hide yes)
+			)
+		)
+		(property "Value" "GND-AUD"
+			(at 59.69 59.944 0)
+			(effects
+				(font
+					(size 1.27 1.27)
+				)
+			)
+		)
+		(property "Footprint" ""
+			(at 59.69 55.88 0)
+			(effects
+				(font
+					(size 1.27 1.27)
+				)
+				(hide yes)
+			)
+		)
+		(property "Datasheet" ""
+			(at 59.69 55.88 0)
+			(effects
+				(font
+					(size 1.27 1.27)
+				)
+				(hide yes)
+			)
+		)
+		(property "Description" "Power symbol creates a global label with name \"GND\" , ground"
+			(at 59.69 55.88 0)
+			(effects
+				(font
+					(size 1.27 1.27)
+				)
+				(hide yes)
+			)
+		)
+		(pin "1"
+		)
+		(instances
+			(project "wb50"
+				(path "/6805e3ef-87bd-473d-890f-05ae2da73c1a/f1b5402f-417b-4ade-9709-94213592078e"
+					(reference "#PWR047")
+					(unit 1)
+				)
+			)
+		)
+	)
+	(symbol
 		(lib_id "Connector:TestPoint_Small")
 		(at 297.18 140.97 0)
@@
 			)
 		)
-		(property "Footprint" "TestPoint:TestPoint_THTPad_D2.0mm_Drill1.0mm"
+		(property "Footprint" "TestPoint:TestPoint_THTPad_D3.0mm_Drill1.5mm"
 			(at 302.26 140.97 0)
 			(effects
@@
 			)
 		)
-		(property "Footprint" "TestPoint:TestPoint_THTPad_D2.0mm_Drill1.0mm"
+		(property "Footprint" "TestPoint:TestPoint_THTPad_D3.0mm_Drill1.5mm"
 			(at 313.69 143.51 0)
 			(effects
@@
 			)
 		)
-		(property "Footprint" "TestPoint:TestPoint_THTPad_D2.0mm_Drill1.0mm"
+		(property "Footprint" "TestPoint:TestPoint_THTPad_D3.0mm_Drill1.5mm"
 			(at 302.26 147.32 0)
 			(effects
@@
 	)
 	(symbol
+		(lib_id "wb50_symbols:NetTie")
+		(at 64.77 53.34 0)
+		(unit 1)
+		(exclude_from_sim no)
+		(in_bom yes)
+		(on_board yes)
+		(dnp no)
+		(fields_autoplaced yes)
+		(property "Reference" "N2"
+			(at 64.77 48.26 0)
+			(effects
+				(font
+					(size 1.27 1.27)
+				)
+			)
+		)
+		(property "Value" "~"
+			(at 64.77 50.8 0)
+			(effects
+				(font
+					(size 1.27 1.27)
+				)
+			)
+		)
+		(property "Footprint" "wb50_footprints:NetTie_0.5mm_2Pad"
+			(at 64.77 53.34 0)
+			(effects
+				(font
+					(size 1.27 1.27)
+				)
+				(hide yes)
+			)
+		)
+		(property "Datasheet" ""
+			(at 64.77 53.34 0)
+			(effects
+				(font
+					(size 1.27 1.27)
+				)
+				(hide yes)
+			)
+		)
+		(property "Description" ""
+			(at 64.77 53.34 0)
+			(effects
+				(font
+					(size 1.27 1.27)
+				)
+				(hide yes)
+			)
+		)
+		(pin "2"
+		)
+		(pin "1"
+		)
+		(instances
+			(project "wb50"
+				(path "/6805e3ef-87bd-473d-890f-05ae2da73c1a/f1b5402f-417b-4ade-9709-94213592078e"
+					(reference "N2")
+					(unit 1)
+				)
+			)
+		)
+	)
+	(symbol
 		(lib_id "jlcpcb:CR1W-10M±5%-6T63")
 		(at 196.85 114.3 270)
@@
 					(unit 1)
 				)
+			)
+		)
+	)
+	(symbol
+		(lib_id "power:GND")
+		(at 72.39 55.88 0)
+		(unit 1)
+		(exclude_from_sim no)
+		(in_bom yes)
+		(on_board yes)
+		(dnp no)
+		(property "Reference" "#PWR048"
+			(at 72.39 62.23 0)
+			(effects
+				(font
+					(size 1.27 1.27)
+				)
+				(hide yes)
+			)
+		)
+		(property "Value" "GND-PWR"
+			(at 72.39 59.944 0)
+			(effects
+				(font
+					(size 1.27 1.27)
+				)
+			)
+		)
+		(property "Footprint" ""
+			(at 72.39 55.88 0)
+			(effects
+				(font
+					(size 1.27 1.27)
+				)
+				(hide yes)
+			)
+		)
+		(property "Datasheet" ""
+			(at 72.39 55.88 0)
+			(effects
+				(font
+					(size 1.27 1.27)
+				)
+				(hide yes)
+			)
+		)
+		(property "Description" "Power symbol creates a global label with name \"GND\" , ground"
+			(at 72.39 55.88 0)
+			(effects
+				(font
+					(size 1.27 1.27)
+				)
+				(hide yes)
+			)
+		)
+		(pin "1"
+		)
+		(instances
+			(project "wb50"
+				(path "/6805e3ef-87bd-473d-890f-05ae2da73c1a/f1b5402f-417b-4ade-9709-94213592078e"
+					(reference "#PWR048")
+					(unit 1)
+				)

Commit message: update design
Parts:
- removed X-BS-1: 1, TestPoint:TestPoint_THTPad_D3.0mm_Drill1.5mm, symbol Connector:TestPoint_Small
- removed X-BS-2: 2, TestPoint:TestPoint_THTPad_D3.0mm_Drill1.5mm, symbol Connector:TestPoint_Small
- removed X-BS-3: 3, TestPoint:TestPoint_THTPad_D3.0mm_Drill1.5mm, symbol Connector:TestPoint_Small
- added U35: MT-0-103-C004-N004-RS, footprints:SW-TH_MT-0-102-C004-N004-RS, symbol symbols:MT-0-103-C004-N004-RS
Connections:
- net at U9.2: now also U35.1
- net at U10.2: now also U35.3
- net at RELAY2.10, RV7.2: now also U35.2
Other:
- note removed: "Bright Switch Solder Points"
Changed lines of the file:
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@@
 	(generator_version "9.0")
 	(paper "A3")
-	(text "Bright Switch\nSolder Points"
-		(exclude_from_sim no)
-		(at 310.896 151.638 0)
-		(effects
-			(font
-				(size 1.27 1.27)
-			)
-		)
-	)
 	(junction
 		(at 152.4 90.17)
@@
 	(wire
 		(pts
-			(xy 293.37 140.97) (xy 297.18 140.97)
-		)
-		(stroke
-			(width 0)
-			(type default)
-		)
-	)
-	(wire
-		(pts
 			(xy 62.23 53.34) (xy 59.69 53.34)
 		)
@@
 	(wire
 		(pts
-			(xy 293.37 147.32) (xy 297.18 147.32)
-		)
-		(stroke
-			(width 0)
-			(type default)
-		)
-	)
-	(wire
-		(pts
 			(xy 179.07 104.14) (xy 196.85 104.14)
 		)
@@
 	(wire
 		(pts
+			(xy 295.91 146.05) (xy 298.45 146.05)
+		)
+		(stroke
+			(width 0)
+			(type default)
+		)
+	)
+	(wire
+		(pts
 			(xy 337.82 138.43) (xy 337.82 134.62)
 		)
@@
 	(wire
 		(pts
+			(xy 293.37 140.97) (xy 298.45 140.97)
+		)
+		(stroke
+			(width 0)
+			(type default)
+		)
+	)
+	(wire
+		(pts
 			(xy 137.16 134.62) (xy 137.16 138.43)
 		)
@@
 	(wire
 		(pts
+			(xy 295.91 147.32) (xy 295.91 146.05)
+		)
+		(stroke
+			(width 0)
+			(type default)
+		)
+	)
+	(wire
+		(pts
 			(xy 68.58 143.51) (xy 68.58 147.32)
 		)
@@
 	(wire
 		(pts
+			(xy 293.37 147.32) (xy 295.91 147.32)
+		)
+		(stroke
+			(width 0)
+			(type default)
+		)
+	)
+	(wire
+		(pts
 			(xy 363.22 124.46) (xy 363.22 138.43)
 		)
@@
 	)
 	(symbol
-		(lib_id "Connector:TestPoint_Small")
-		(at 297.18 140.97 0)
-		(unit 1)
-		(exclude_from_sim no)
-		(in_bom yes)
-		(on_board yes)
-		(dnp no)
-		(fields_autoplaced yes)
-		(property "Reference" "X-BS-3"
-			(at 298.45 139.6999 0)
-			(effects
-				(font
-					(size 1.27 1.27)
-				)
-				(justify left)
-			)
-		)
-		(property "Value" "3"
-			(at 298.45 142.2399 0)
-			(effects
-				(font
-					(size 1.27 1.27)
-				)
-				(justify left)
-			)
-		)
-		(property "Footprint" "TestPoint:TestPoint_THTPad_D3.0mm_Drill1.5mm"
-			(at 302.26 140.97 0)
-			(effects
-				(font
-					(size 1.27 1.27)
-				)
-				(hide yes)
-			)
-		)
-		(property "Datasheet" "~"
-			(at 302.26 140.97 0)
-			(effects
-				(font
-					(size 1.27 1.27)
-				)
-				(hide yes)
-			)
-		)
-		(property "Description" "test point"
-			(at 297.18 140.97 0)
-			(effects
-				(font
-					(size 1.27 1.27)
-				)
-				(hide yes)
-			)
-		)
-		(pin "1"
-		)
-		(instances
-			(project ""
-				(path "/6805e3ef-87bd-473d-890f-05ae2da73c1a/f1b5402f-417b-4ade-9709-94213592078e"
-					(reference "X-BS-3")
-					(unit 1)
-				)
-			)
-		)
-	)
-	(symbol
 		(lib_id "power:GND")
 		(at 74.93 147.32 0)
@@
 		(dnp no)
 		(property "Reference" "U9"
-			(at 287.274 135.636 0)
+			(at 285.242 134.874 0)
 			(effects
 				(font
@@
 		)
 		(property "Value" "500pF 500V 5%"
-			(at 281.432 137.668 0)
+			(at 279.4 137.414 0)
 			(effects
 				(font
@@
 	)
 	(symbol
-		(lib_id "Connector:TestPoint_Small")
-		(at 308.61 143.51 0)
-		(unit 1)
-		(exclude_from_sim no)
-		(in_bom yes)
-		(on_board yes)
-		(dnp no)
-		(fields_autoplaced yes)
-		(property "Reference" "X-BS-2"
-			(at 309.88 142.2399 0)
-			(effects
-				(font
-					(size 1.27 1.27)
-				)
-				(justify left)
-			)
-		)
-		(property "Value" "2"
-			(at 309.88 144.7799 0)
-			(effects
-				(font
-					(size 1.27 1.27)
-				)
-				(justify left)
-			)
-		)
-		(property "Footprint" "TestPoint:TestPoint_THTPad_D3.0mm_Drill1.5mm"
-			(at 313.69 143.51 0)
-			(effects
-				(font
-					(size 1.27 1.27)
-				)
-				(hide yes)
-			)
-		)
-		(property "Datasheet" "~"
-			(at 313.69 143.51 0)
-			(effects
-				(font
-					(size 1.27 1.27)
-				)
-				(hide yes)
-			)
-		)
-		(property "Description" "test point"
-			(at 308.61 143.51 0)
-			(effects
-				(font
-					(size 1.27 1.27)
-				)
-				(hide yes)
-			)
-		)
-		(pin "1"
-		)
-		(instances
-			(project "wb50"
-				(path "/6805e3ef-87bd-473d-890f-05ae2da73c1a/f1b5402f-417b-4ade-9709-94213592078e"
-					(reference "X-BS-2")
-					(unit 1)
-				)
-			)
-		)
-	)
-	(symbol
 		(lib_id "Device:R_Potentiometer")
 		(at 294.64 104.14 0)
@@
 	)
 	(symbol
-		(lib_id "Connector:TestPoint_Small")
-		(at 297.18 147.32 0)
-		(unit 1)
-		(exclude_from_sim no)
-		(in_bom yes)
-		(on_board yes)
-		(dnp no)
-		(fields_autoplaced yes)
-		(property "Reference" "X-BS-1"
-			(at 298.45 146.0499 0)
-			(effects
-				(font
-					(size 1.27 1.27)
-				)
-				(justify left)
-			)
-		)
-		(property "Value" "1"
-			(at 298.45 148.5899 0)
-			(effects
-				(font
-					(size 1.27 1.27)
-				)
-				(justify left)
-			)
-		)
-		(property "Footprint" "TestPoint:TestPoint_THTPad_D3.0mm_Drill1.5mm"
-			(at 302.26 147.32 0)
-			(effects
-				(font
-					(size 1.27 1.27)
-				)
-				(hide yes)
-			)
-		)
-		(property "Datasheet" "~"
-			(at 302.26 147.32 0)
-			(effects
-				(font
-					(size 1.27 1.27)
-				)
-				(hide yes)
-			)
-		)
-		(property "Description" "test point"
-			(at 297.18 147.32 0)
-			(effects
-				(font
-					(size 1.27 1.27)
-				)
-				(hide yes)
-			)
-		)
-		(pin "1"
-		)
-		(instances
-			(project "wb50"
-				(path "/6805e3ef-87bd-473d-890f-05ae2da73c1a/f1b5402f-417b-4ade-9709-94213592078e"
-					(reference "X-BS-1")
-					(unit 1)
-				)
-			)
-		)
-	)
-	(symbol
 		(lib_id "power:+12V")
 		(at 152.4 82.55 0)
@@
 					(unit 1)
 				)
+			)
+		)
+	)
+	(symbol
+		(lib_id "symbols:MT-0-103-C004-N004-RS")
+		(at 303.53 143.51 0)
+		(mirror y)
+		(unit 1)
+		(exclude_from_sim no)
+		(in_bom yes)
+		(on_board yes)
+		(dnp no)
+		(property "Reference" "U35"
+			(at 304.8 135.636 0)
+			(effects
+				(font
+					(size 1.27 1.27)
+				)
+			)
+		)
+		(property "Value" "MT-0-103-C004-N004-RS"
+			(at 310.896 138.176 0)
+			(effects
+				(font
+					(size 1.27 1.27)
+				)
+			)
+		)
+		(property "Footprint" "footprints:SW-TH_MT-0-102-C004-N004-RS"
+			(at 303.53 153.67 0)
+			(effects
+				(font
+					(size 1.27 1.27)
+					(italic yes)
+				)
+				(hide yes)
+			)
+		)
+		(property "Datasheet" "https://item.szlcsc.com/1879287.html"
+			(at 305.816 143.383 0)
+			(effects
+				(font
+					(size 1.27 1.27)
+				)
+				(justify left)
+				(hide yes)
+			)
+		)
+		(property "Description" ""
+			(at 303.53 143.51 0)
+			(effects
+				(font
+					(size 1.27 1.27)
+				)
+				(hide yes)
+			)
+		)
+		(property "LCSC" "C22448931"
+			(at 303.53 143.51 0)
+			(effects
+				(font
+					(size 1.27 1.27)
+				)
+				(hide yes)
+			)
+		)
+		(pin "5"
+		)
+		(pin "1"
+		)
+		(pin "3"
+		)
+		(pin "2"
+		)
+		(pin "4"
+		)
+		(instances
+			(project ""
+				(path "/6805e3ef-87bd-473d-890f-05ae2da73c1a/f1b5402f-417b-4ade-9709-94213592078e"
+					(reference "U35")
+					(unit 1)
+				)
