File: electronics/main/schematics/power.kicad_sch (KiCad schematic)
At the start: 28 parts, among them U31 16A 20mm 500V 5mm Plugin Fuse, U32 CR2W-4K7±5%-9T73, U33 3314G-1-503E

Commit message: schematic  checked!
Connections:
- net Bias-Set: now also C13.2; no longer C13.1
- net GND-PWR: now also C13.1, C14.1; no longer C13.2, C14.2
- net at D3.2 (A), R29.2: now also C14.2; no longer C14.1
Other:
- note added: "Kopplungssimulation"

Commit message: updated PCB
Parts:
- AC-IN1, AC-IN2, AC-IN3: footprint TestPoint:TestPoint_THTPad_D2.0mm_Drill1.0mm -> TestPoint:TestPoint_THTPad_D3.0mm_Drill1.5mm
- AC-IN6, AC-IN7, AC-IN8: footprint TestPoint:TestPoint_THTPad_D2.0mm_Drill1.0mm -> TestPoint:TestPoint_THTPad_D4.0mm_Drill2.0mm
- Choke1, Choke2: footprint TestPoint:TestPoint_THTPad_D2.0mm_Drill1.0mm -> TestPoint:TestPoint_THTPad_D2.5mm_Drill1.2mm
Connections:
- net GND-PWR: no longer C10.2, C11.2, C12.2, C9.2
- new net GND-AUD: C10.2, C11.2, C12.2, C9.2

Commit message: update design
Parts:
- added GND-AUD1, HV-B1: 1, TestPoint:TestPoint_THTPad_D3.0mm_Drill1.5mm, symbol Connector:TestPoint_Small
Connections:
- net GND-AUD: now also GND-AUD1.1
- net HV-B: now also HV-B1.1
Changed lines of the file:
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@@
 	(wire
 		(pts
+			(xy 137.16 68.58) (xy 137.16 88.9)
+		)
+		(stroke
+			(width 0)
+			(type default)
+		)
+	)
+	(wire
+		(pts
 			(xy 137.16 88.9) (xy 144.78 88.9)
 		)
@@
 	)
 	(symbol
+		(lib_id "power:GND")
+		(at 148.59 68.58 0)
+		(unit 1)
+		(exclude_from_sim no)
+		(in_bom yes)
+		(on_board yes)
+		(dnp no)
+		(fields_autoplaced yes)
+		(property "Reference" "#PWR052"
+			(at 148.59 74.93 0)
+			(effects
+				(font
+					(size 1.27 1.27)
+				)
+				(hide yes)
+			)
+		)
+		(property "Value" "GND-AUD"
+			(at 148.59 73.66 0)
+			(effects
+				(font
+					(size 1.27 1.27)
+				)
+			)
+		)
+		(property "Footprint" ""
+			(at 148.59 68.58 0)
+			(effects
+				(font
+					(size 1.27 1.27)
+				)
+				(hide yes)
+			)
+		)
+		(property "Datasheet" ""
+			(at 148.59 68.58 0)
+			(effects
+				(font
+					(size 1.27 1.27)
+				)
+				(hide yes)
+			)
+		)
+		(property "Description" "Power symbol creates a global label with name \"GND\" , ground"
+			(at 148.59 68.58 0)
+			(effects
+				(font
+					(size 1.27 1.27)
+				)
+				(hide yes)
+			)
+		)
+		(pin "1"
+		)
+		(instances
+			(project "wb50"
+				(path "/6805e3ef-87bd-473d-890f-05ae2da73c1a/1d95444c-de5c-440e-b338-1d9c97a29411"
+					(reference "#PWR052")
+					(unit 1)
+				)
+			)
+		)
+	)
+	(symbol
 		(lib_id "jlcpcb:LKML2502H330MF")
 		(at 137.16 96.52 0)
@@
 	)
 	(symbol
+		(lib_id "Connector:TestPoint_Small")
+		(at 137.16 68.58 90)
+		(unit 1)
+		(exclude_from_sim no)
+		(in_bom yes)
+		(on_board yes)
+		(dnp no)
+		(fields_autoplaced yes)
+		(property "Reference" "HV-B1"
+			(at 137.16 63.5 90)
+			(effects
+				(font
+					(size 1.27 1.27)
+				)
+			)
+		)
+		(property "Value" "1"
+			(at 137.16 66.04 90)
+			(effects
+				(font
+					(size 1.27 1.27)
+				)
+			)
+		)
+		(property "Footprint" "TestPoint:TestPoint_THTPad_D3.0mm_Drill1.5mm"
+			(at 137.16 63.5 0)
+			(effects
+				(font
+					(size 1.27 1.27)
+				)
+				(hide yes)
+			)
+		)
+		(property "Datasheet" "~"
+			(at 137.16 63.5 0)
+			(effects
+				(font
+					(size 1.27 1.27)
+				)
+				(hide yes)
+			)
+		)
+		(property "Description" "test point"
+			(at 137.16 68.58 0)
+			(effects
+				(font
+					(size 1.27 1.27)
+				)
+				(hide yes)
+			)
+		)
+		(pin "1"
+		)
+		(instances
+			(project "wb50"
+				(path "/6805e3ef-87bd-473d-890f-05ae2da73c1a/1d95444c-de5c-440e-b338-1d9c97a29411"
+					(reference "HV-B1")
+					(unit 1)
+				)
+			)
+		)
+	)
+	(symbol
 		(lib_id "power:GND")
 		(at 179.07 153.67 0)
@@
 					(unit 1)
 				)
+			)
+		)
+	)
+	(symbol
+		(lib_id "Connector:TestPoint_Small")
+		(at 148.59 68.58 90)
+		(unit 1)
+		(exclude_from_sim no)
+		(in_bom yes)
+		(on_board yes)
+		(dnp no)
+		(fields_autoplaced yes)
+		(property "Reference" "GND-AUD1"
+			(at 148.59 63.5 90)
+			(effects
+				(font
+					(size 1.27 1.27)
+				)
+			)
+		)
+		(property "Value" "1"
+			(at 148.59 66.04 90)
+			(effects
+				(font
+					(size 1.27 1.27)
+				)
+			)
+		)
+		(property "Footprint" "TestPoint:TestPoint_THTPad_D3.0mm_Drill1.5mm"
+			(at 148.59 63.5 0)
+			(effects
+				(font
+					(size 1.27 1.27)
+				)
+				(hide yes)
+			)
+		)
+		(property "Datasheet" "~"
+			(at 148.59 63.5 0)
+			(effects
+				(font
+					(size 1.27 1.27)
+				)
+				(hide yes)
+			)
+		)
+		(property "Description" "test point"
+			(at 148.59 68.58 0)
+			(effects
+				(font
+					(size 1.27 1.27)
+				)
+				(hide yes)
+			)
+		)
+		(pin "1"
+		)
+		(instances
+			(project "wb50"
+				(path "/6805e3ef-87bd-473d-890f-05ae2da73c1a/1d95444c-de5c-440e-b338-1d9c97a29411"
+					(reference "GND-AUD1")
+					(unit 1)
+				)

Commit message: add fx loop, add new shield
Parts:
- added C15: 18uF 450V ±20%, footprints:CAP-TH_BD10.0-P5.00-D1.0-FD, symbol jlcpcb:18uF_450V
- added R43: CF2W-2200Ω±5%_T, footprints:RES-TH_BD5.5-L15.0-P19.00-D0.8, symbol symbols:CF2W-2200Ω±5%_T
Connections:
- net GND-AUD: now also C15.2
- net HV-B: now also R43.1
- new net HV-F: C15.1, R43.2
