File: electronics/main/wb50.kicad_pcb (KiCad board)
At the start: 6 copper layers, 405 x 100 mm, 15 parts, among them J1 IN, J2 SW

Commit message: update aux voltage
Parts:
- added C1: VKME1002C220MV, footprints:CAP-SMD_BD10.0-L10.3-W10.3-LS11.7-FD, F.Cu at (461.2, 183.2)
- added C2: LKMI2501C682MF, footprints:CAP-TH_BD16.0-P7.50-D1.2-FD, F.Cu at (502.0, 216.2)
- added C3: CC0805KRX7R9BB104, footprints:C0805, F.Cu at (504.0, 192.4)
- added C4: CC0805KRX7R9BB104, footprints:C0805, F.Cu at (501.5, 181.4)
- added MH1: TestPoint, MountingHole:MountingHole_2.2mm_M2_DIN965_Pad_TopBottom, F.Cu at (490.0, 189.4)
- added MH2: TestPoint, MountingHole:MountingHole_2.2mm_M2_DIN965_Pad_TopBottom, F.Cu at (515.5, 189.4)
- added U1: XSD366-094, footprints:HEATSINK-TH_XSD366-094, F.Cu at (502.8, 189.4)
- added U2: L7812CV-DG, footprints:TO-220-3_L10.0-W4.5-P2.54-L, F.Cu at (502.8, 186.3)
- added U3: AB24S, footprints:ABS-SMD_L5.0-W4.4-P4.00-LS7.0-BL, F.Cu at (515.8, 211.4)
- added X1: 345V - Lila, TestPoint:TestPoint_THTPad_D3.0mm_Drill1.5mm, F.Cu at (181.8, 138.7)
- added X2: CT_HV - Grau, TestPoint:TestPoint_THTPad_D3.0mm_Drill1.5mm, F.Cu at (181.8, 143.8)
- added X3: 345V - Lila, TestPoint:TestPoint_THTPad_D3.0mm_Drill1.5mm, F.Cu at (186.9, 138.7)
- added X4: 3.13V - Grün, TestPoint:TestPoint_THTPad_D3.0mm_Drill1.5mm, F.Cu at (186.9, 143.8)
- added X5: CT_HEAT - Schwarz, TestPoint:TestPoint_THTPad_D3.0mm_Drill1.5mm, F.Cu at (191.9, 138.7)
- added X6: 3.13V - Grün, TestPoint:TestPoint_THTPad_D3.0mm_Drill1.5mm, F.Cu at (191.9, 143.8)
- added X7: 12,6V - Rot, TestPoint:TestPoint_THTPad_D3.0mm_Drill1.5mm, F.Cu at (520.8, 205.0)
- added X8: 0V - Rot, TestPoint:TestPoint_THTPad_D3.0mm_Drill1.5mm, F.Cu at (520.8, 218.0)

Commit message: PI stage ready
Parts:
- moved X1 67.3 mm to (134.4, 186.4)
- moved X2 67.3 mm to (134.4, 191.5)
- moved X3 67.3 mm to (139.5, 186.4)
- moved X4 67.3 mm to (139.5, 191.5)
- moved X5 67.3 mm to (144.6, 186.4)
- moved X6 67.3 mm to (144.6, 191.5)
Other:
- board size 405 x 100 mm -> 405 x 190 mm
Changed lines of the file:
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@@
 	(footprint "TestPoint:TestPoint_THTPad_D3.0mm_Drill1.5mm"
 		(layer "F.Cu")
-		(at 181.85 138.7)
+		(at 134.45 186.45)
 		(descr "THT pad as test Point, diameter 3.0mm, hole diameter 1.5mm")
 		(tags "test point THT pad")
@@
 	(footprint "TestPoint:TestPoint_THTPad_D3.0mm_Drill1.5mm"
 		(layer "F.Cu")
-		(at 191.95 143.75)
+		(at 144.55 191.5)
 		(descr "THT pad as test Point, diameter 3.0mm, hole diameter 1.5mm")
 		(tags "test point THT pad")
@@
 	(footprint "TestPoint:TestPoint_THTPad_D3.0mm_Drill1.5mm"
 		(layer "F.Cu")
-		(at 186.9 143.75)
+		(at 139.5 191.5)
 		(descr "THT pad as test Point, diameter 3.0mm, hole diameter 1.5mm")
 		(tags "test point THT pad")
@@
 	(footprint "TestPoint:TestPoint_THTPad_D3.0mm_Drill1.5mm"
 		(layer "F.Cu")
-		(at 181.85 143.75)
+		(at 134.45 191.5)
 		(descr "THT pad as test Point, diameter 3.0mm, hole diameter 1.5mm")
 		(tags "test point THT pad")
@@
 	(footprint "TestPoint:TestPoint_THTPad_D3.0mm_Drill1.5mm"
 		(layer "F.Cu")
-		(at 186.9 138.7)
+		(at 139.5 186.45)
 		(descr "THT pad as test Point, diameter 3.0mm, hole diameter 1.5mm")
 		(tags "test point THT pad")
@@
 	(footprint "TestPoint:TestPoint_THTPad_D3.0mm_Drill1.5mm"
 		(layer "F.Cu")
-		(at 191.95 138.7)
+		(at 144.55 186.45)
 		(descr "THT pad as test Point, diameter 3.0mm, hole diameter 1.5mm")
 		(tags "test point THT pad")
@@
 		)
 	)
-	(gr_rect
-		(start 119.5 176)
+	(gr_arc
+		(start 367.5 176)
+		(mid 366.085786 175.414214)
+		(end 365.5 174)
+		(stroke
+			(width 0.2)
+			(type default)
+		)
+		(locked yes)
+		(layer "Edge.Cuts")
+	)
+	(gr_line
+		(start 524.5 176)
 		(end 524.5 276)
 		(stroke
@@
 			(type default)
 		)
-		(fill no)
+		(locked yes)
+		(layer "Edge.Cuts")
+	)
+	(gr_line
+		(start 524.5 276)
+		(end 119.5 276)
+		(stroke
+			(width 0.2)
+			(type default)
+		)
+		(locked yes)
+		(layer "Edge.Cuts")
+	)
+	(gr_line
+		(start 365.5 174)
+		(end 365.5 86)
+		(stroke
+			(width 0.2)
+			(type default)
+		)
+		(locked yes)
+		(layer "Edge.Cuts")
+	)
+	(gr_line
+		(start 213.5 86)
+		(end 365.5 86)
+		(stroke
+			(width 0.2)
+			(type default)
+		)
+		(locked yes)
+		(layer "Edge.Cuts")
+	)
+	(gr_arc
+		(start 213.5 174)
+		(mid 212.914214 175.414214)
+		(end 211.5 176)
+		(stroke
+			(width 0.2)
+			(type default)
+		)
+		(locked yes)
+		(layer "Edge.Cuts")
+	)
+	(gr_line
+		(start 367.5 176)
+		(end 524.5 176)
+		(stroke
+			(width 0.2)
+			(type default)
+		)
+		(locked yes)
+		(layer "Edge.Cuts")
+	)
+	(gr_line
+		(start 119.5 176)
+		(end 211.5 176)
+		(stroke
+			(width 0.2)
+			(type default)
+		)
+		(locked yes)
+		(layer "Edge.Cuts")
+	)
+	(gr_line
+		(start 119.5 276)
+		(end 119.5 176)
+		(stroke
+			(width 0.2)
+			(type default)
+		)
+		(locked yes)
+		(layer "Edge.Cuts")
+	)
+	(gr_line
+		(start 213.5 174)
+		(end 213.5 86)
+		(stroke
+			(width 0.2)
+			(type default)
+		)
 		(locked yes)
 		(layer "Edge.Cuts")

Commit message: schematic ready? - check
Parts:
- added Audio-To-FX1: 1, TestPoint:TestPoint_THTPad_D2.0mm_Drill1.0mm, F.Cu at (154.3, 64.9)
- added Audo-From-FX1: 1, TestPoint:TestPoint_THTPad_D2.0mm_Drill1.0mm, F.Cu at (154.3, 68.9)
- added C5: 0,82uF 400V 20 %, footprints:CAP-TH_BD6.3-P2.50-D1.0-FD, F.Cu at (96.3, 130.5)
- added C6: 0,82uF 400V 20 %, footprints:CAP-TH_BD6.3-P2.50-D1.0-FD, F.Cu at (96.3, 138.0)
- added C7: 22uF_450V_16*20, footprints:CAP-TH_BD16.0-P7.50-D1.2-FD, F.Cu at (127.0, 63.6)
- added J3: OUT1, wb50_footprints:WB50_Jack_TRS_6pin_16.2mm, F.Cu at (312.8, 98.2)
- added J4: OUT2, wb50_footprints:WB50_Jack_TRS_6pin_16.2mm, F.Cu at (345.2, 98.2)
- added R1: 33k 500V 2W, footprints:RES-TH_BD3.0-L9.5-P13.50-D0.6, F.Cu at (68.8, 145.6)
- added R10: CR1/2WS-470K±5%-ST52, footprints:RES-TH_BD2.7-L6.2-P10.20-D0.4, F.Cu at (158.6, 56.9)
- added R11: CR1/2WS-470K±5%-ST52, footprints:RES-TH_BD2.7-L6.2-P10.20-D0.4, F.Cu at (158.6, 60.9)
- added R12: CR1W-100K±5%-TT63, footprints:RES-TH_BD4.5-L11.0-P15.00-D0.7, F.Cu at (155.4, 37.7)
- added R13: 820R 350V 500mW, footprints:RES-TH_BD4.0-L10.5-P14.50-D0.6, F.Cu at (155.2, 49.0)
- added R14: CR1W-100K±5%-TT63, footprints:RES-TH_BD4.5-L11.0-P15.00-D0.7, F.Cu at (155.4, 43.5)
- added R15: 33k 500V 2W, footprints:RES-TH_BD3.0-L9.5-P13.50-D0.6, F.Cu at (143.8, 76.5)
- added R16: CR1W-10M±5%-6T63, footprints:RES-TH_BD4.5-L11.0-P15.00-D0.7, F.Cu at (97.7, 79.3)
- added R17: 1Meg 500V 250mW, footprints:RES-TH_BD2.4-L6.3-P10.30-D0.6, F.Cu at (110.0, 40.6)
- added R18: 1Meg 500V 250mW, footprints:RES-TH_BD2.4-L6.3-P10.30-D0.6, F.Cu at (110.0, 44.3)
- added R19: CF3WS-10KΩ±5%_T, footprints:RES-TH_BD5.5-L15.0-P19.00-D0.8, F.Cu at (99.6, 67.8)
- added R2: 1Meg 500V 250mW, footprints:RES-TH_BD2.4-L6.3-P10.30-D0.6, F.Cu at (84.7, 146.3)
- added R20: CR1W-100K±5%-TT63, footprints:RES-TH_BD4.5-L11.0-P15.00-D0.7, F.Cu at (97.7, 85.0)
- added R21: CR1/4W-47K±5%-ST52, footprints:RES-TH_BD2.7-L6.2-P10.20-D0.4, F.Cu at (110.0, 36.8)
- added R22: CFR-25JT-52-1K5, footprints:RES-TH_BD2.4-L6.3-P10.30-D0.6, F.Cu at (140.1, 107.4)
- added R23: CFR-25JT-52-1K5, footprints:RES-TH_BD2.4-L6.3-P10.30-D0.6, F.Cu at (140.1, 111.0)
- added R3: CR1W-100K±5%-TT63, footprints:RES-TH_BD4.5-L11.0-P15.00-D0.7, F.Cu at (69.5, 123.3)
- added R4: CR1/4W-2K7±5%-ST26, footprints:RES-TH_BD2.7-L6.2-P10.20-D0.4, F.Cu at (98.8, 143.8)
- added R5: CR1W-100K±5%-TT63, footprints:RES-TH_BD4.5-L11.0-P15.00-D0.7, F.Cu at (69.5, 129.1)
- added R6: 33k 500V 2W, footprints:RES-TH_BD3.0-L9.5-P13.50-D0.6, F.Cu at (68.8, 149.8)
- added R7: CR1W-10M±5%-6T63, footprints:RES-TH_BD4.5-L11.0-P15.00-D0.7, F.Cu at (69.5, 134.8)
- added R8: CR1/4W-2K7±5%-ST26, footprints:RES-TH_BD2.7-L6.2-P10.20-D0.4, F.Cu at (98.8, 147.7)
- added R9: CR1W-100K±5%-TT63, footprints:RES-TH_BD4.5-L11.0-P15.00-D0.7, F.Cu at (69.5, 140.6)
- added RELAY1: G5V-1-12V, footprints:RELAY-TH_G5V-1, F.Cu at (85.5, 131.2)
- added RELAY2: G5V-1-12V, footprints:RELAY-TH_G5V-1, F.Cu at (85.5, 140.1)
- added RELAY3: G5V-1-12V, footprints:RELAY-TH_G5V-1, F.Cu at (125.4, 76.7)
- added U10: 250pF 500V 5%, wb50_footprints:MICA_CAP_L15.5_W3.6_P8.7, F.Cu at (97.2, 112.5)
- added U11: 500pF 500V 5%, wb50_footprints:MICA_CAP_L15.5_W3.6_P8.7, F.Cu at (143.9, 57.4)
- added U12: 500pF 500V 5%, wb50_footprints:MICA_CAP_L15.5_W3.6_P8.7, F.Cu at (143.9, 62.2)
- added U13: 500pF 500V 5%, wb50_footprints:MICA_CAP_L15.5_W3.6_P8.7, F.Cu at (143.9, 67.1)
- added U14: 22n 630V 5%, wb50_footprints:MUSTARD_CAP_D8.5_L20.5_P25.5, F.Cu at (132.4, 39.9)
- added U15: 22n 630V 5%, wb50_footprints:MUSTARD_CAP_D8.5_L20.5_P25.5, F.Cu at (132.4, 49.9)
- added U16: 500pF 500V 5%, wb50_footprints:MICA_CAP_L15.5_W3.6_P8.7, F.Cu at (143.9, 71.9)
- added U17: 22n 630V 5%, wb50_footprints:MUSTARD_CAP_D8.5_L20.5_P25.5, F.Cu at (74.7, 63.2)
- added U18: 470R 500V 2W, footprints:RES-TH_BD5.0-L15.5-P19.50-D0.7, F.Cu at (100.2, 61.3)
- added U19: 100n 630V 5%, wb50_footprints:MUSTARD_CAP_D10_L32_P40.4, F.Cu at (82.2, 40.7)
- added U20: CF2WS-82KΩ±5%_T, footprints:RES-TH_BD4.0-L11.5-P15.50-D0.7, F.Cu at (97.8, 73.8)
- added U21: 100pF 500V 5%, wb50_footprints:MICA_CAP_L15.5_W3.6_P8.7, F.Cu at (97.2, 90.3)
- added U22: CR1/2W-220K±5%-XT52, footprints:RES-TH_BD3.5-L9.0-P13.00-D0.5, F.Cu at (96.6, 95.1)
- added U23: 100n 630V 5%, wb50_footprints:MUSTARD_CAP_D10_L32_P40.4, F.Cu at (82.2, 52.3)
- added U24: 4n7 630V 5%, wb50_footprints:MUSTARD_CAP_D8.5_L20.5_P25.5, F.Cu at (74.7, 73.2)
- added U25: 22n 630V 5%, wb50_footprints:MUSTARD_CAP_D8.5_L20.5_P25.5, F.Cu at (74.7, 83.3)
- added U26: 22n 630V 5%, wb50_footprints:MUSTARD_CAP_D8.5_L20.5_P25.5, F.Cu at (74.7, 93.3)
- added U27: CR1/2W-220K±5%-XT52, footprints:RES-TH_BD3.5-L9.0-P13.00-D0.5, F.Cu at (126.1, 108.0)
- added U28: CR1/2W-220K±5%-XT52, footprints:RES-TH_BD3.5-L9.0-P13.00-D0.5, F.Cu at (126.1, 112.8)
- added U29: CR-L5W-1KΩJ, footprints:RES-TH_BD9.5-L22.0-P26.00-D0.7, F.Cu at (137.4, 88.7)
- added U30: CR-L5W-1KΩJ, footprints:RES-TH_BD9.5-L22.0-P26.00-D0.7, F.Cu at (137.4, 99.9)
- added U4: CR1/2W-220K±5%-XT52, footprints:RES-TH_BD3.5-L9.0-P13.00-D0.5, F.Cu at (96.6, 117.3)
- added U5: CR2W-68K±5%-9T73, footprints:RES-TH_BD5.0-L15.5-P19.50-D0.7, F.Cu at (89.8, 123.6)
- added U6: 500pF 500V 5%, wb50_footprints:MICA_CAP_L15.5_W3.6_P8.7, F.Cu at (97.2, 102.8)
- added U7: 4n7 630V 5%, wb50_footprints:MUSTARD_CAP_D8.5_L20.5_P25.5, F.Cu at (74.7, 105.4)
- added U8: 2n2 630V 5%, wb50_footprints:MUSTARD_CAP_D8.5_L20.5_P25.5, F.Cu at (74.7, 115.4)
- added U9: 500pF 500V 5%, wb50_footprints:MICA_CAP_L15.5_W3.6_P8.7, F.Cu at (97.2, 107.6)
- added X-BS-1: 1, TestPoint:TestPoint_THTPad_D2.0mm_Drill1.0mm, F.Cu at (102.1, 128.7)
- added X-BS-2: 2, TestPoint:TestPoint_THTPad_D2.0mm_Drill1.0mm, F.Cu at (102.1, 132.8)
- added X-BS-3: 3, TestPoint:TestPoint_THTPad_D2.0mm_Drill1.0mm, F.Cu at (102.1, 136.8)
- added X12: GND_OT, TestPoint:TestPoint_THTPad_D4.0mm_Drill2.0mm, F.Cu at (143.9, 126.2)
- added X9: Audio IN, TestPoint:TestPoint_THTPad_D4.0mm_Drill2.0mm, F.Cu at (143.9, 120.2)
- C1: value VKME1002C220MV -> 33uF 50V; footprint footprints:CAP-SMD_BD10.0-L10.3-W10.3-LS11.7-FD -> footprints:CAP-TH_BD5.0-P2.00-D0.8-FD
- moved C1 5.77 mm to (455.5, 183.8)
Connections:
- C1 pad 1: Net-(U2-OUTPUT) -> +12V
- C4 pad 1: Net-(U2-OUTPUT) -> +12V
- J1 pad 1: unconnected-(J1-Pad1) -> GND-AUD
- J1 pad 2: unconnected-(J1-Pad2) -> /Connectors/Audio_IN
- J1 pad 3: unconnected-(J1-Pad3) -> /Connectors/Audio_IN
- J1 pad 4: unconnected-(J1-Pad4) -> GND-AUD
- J1 pad 5: unconnected-(J1-Pad5) -> GND-AUD
- J1 pad 6: unconnected-(J1-Pad6) -> GND-AUD
- RV1 pad 1: unconnected-(RV1-Pad1) -> Net-(R19-Pad2)
- RV1 pad 2: unconnected-(RV1-Pad2) -> Net-(RV1-Pad2)
- RV1 pad 3: unconnected-(RV1-Pad3) -> GND-AUD
- RV2 pad 1: unconnected-(RV2-Pad1) -> Net-(RV2-Pad1)
- RV2 pad 2: unconnected-(RV2-Pad2) -> Net-(RV2-Pad2)
- RV2 pad 3: unconnected-(RV2-Pad3) -> Net-(RV2-Pad2)
- RV3 pad 1: unconnected-(RV3-Pad1) -> GND-AUD
- RV3 pad 2: unconnected-(RV3-Pad2) -> Net-(RV3-Pad2)
- RV3 pad 3: unconnected-(RV3-Pad3) -> Net-(RV2-Pad1)
- RV4 pad 1: unconnected-(RV4-Pad1) -> Net-(RV2-Pad2)
- RV4 pad 2: unconnected-(RV4-Pad2) -> Net-(Audio-To-FX1-Pad1)
- RV4 pad 3: unconnected-(RV4-Pad3) -> Net-(RV4-Pad3)
- RV5 pad 1: unconnected-(RV5-Pad1) -> Net-(Audo-From-FX1-Pad1)
- RV5 pad 2: unconnected-(RV5-Pad2) -> Net-(RELAY3-Pad10)
- RV5 pad 3: unconnected-(RV5-Pad3) -> GND-AUD
- RV6 pad 1: unconnected-(RV6-Pad1) -> Net-(Audo-From-FX1-Pad1)
- RV6 pad 2: unconnected-(RV6-Pad2) -> Net-(RELAY3-Pad1)
- RV6 pad 3: unconnected-(RV6-Pad3) -> GND-AUD
- RV7 pad 1: unconnected-(RV7-Pad1) -> GND-AUD
- RV7 pad 2: unconnected-(RV7-Pad2) -> Net-(RELAY2-Pad10)
- RV7 pad 3: unconnected-(RV7-Pad3) -> Net-(RV7-Pad3)
- RV8 pad 1: unconnected-(RV8-Pad1) -> GND-AUD
- RV8 pad 2: unconnected-(RV8-Pad2) -> Net-(RELAY2-Pad1)
- RV8 pad 3: unconnected-(RV8-Pad3) -> Net-(RV7-Pad3)
- U2 pad 3: Net-(U2-OUTPUT) -> +12V
- V1 pad 1: unconnected-(V1A-A/P-Pad1) -> Net-(V1A-A/P)
- V1 pad 2: unconnected-(V1A-G-Pad2) -> Net-(V1A-G)
- V1 pad 3: unconnected-(V1A-C/K-Pad3) -> Net-(V1A-C/K)
- V1 pad 4: unconnected-(V1C-H1-Pad4) -> +12V
- V1 pad 5: unconnected-(V1C-H2-Pad5) -> GND-AUX
- V1 pad 6: unconnected-(V1B-A/P-Pad6) -> Net-(V1B-A/P)
- V1 pad 7: unconnected-(V1B-G-Pad7) -> Net-(V1B-G)
- V1 pad 8: unconnected-(V1B-C/K-Pad8) -> Net-(V1B-C/K)
- V2 pad 1: unconnected-(V2A-A/P-Pad1) -> Net-(V2A-A/P)
- V2 pad 2: unconnected-(V2A-G-Pad2) -> Net-(V2A-G)
- V2 pad 3: unconnected-(V2A-C/K-Pad3) -> Net-(V2A-C/K)
- V2 pad 4: unconnected-(V2C-H1-Pad4) -> +12V
- V2 pad 5: unconnected-(V2C-H2-Pad5) -> GND-AUX
- V2 pad 6: unconnected-(V2B-A/P-Pad6) -> HV-D
- V2 pad 7: unconnected-(V2B-G-Pad7) -> Net-(V2A-A/P)
- V2 pad 8: unconnected-(V2B-C/K-Pad8) -> Net-(V2B-C/K)
- V3 pad 1: unconnected-(V3A-A/P-Pad1) -> Net-(V3A-A/P)
- V3 pad 2: unconnected-(V3A-G-Pad2) -> Net-(V3A-G)
- V3 pad 3: unconnected-(V3A-C/K-Pad3) -> Net-(V3A-C/K)
- V3 pad 4: unconnected-(V3C-H1-Pad4) -> +12V
- V3 pad 5: unconnected-(V3C-H2-Pad5) -> GND-AUX
- V3 pad 6: unconnected-(V3B-A/P-Pad6) -> Net-(V3B-A/P)
- V3 pad 7: unconnected-(V3B-G-Pad7) -> Net-(V3B-G)
- V3 pad 8: unconnected-(V3B-C/K-Pad8) -> Net-(V3A-C/K)
- V4 pad 1: unconnected-(V4A-g3-Pad1) -> GND-AUD
- V4 pad 4: unconnected-(V4A-g2-Pad4) -> Net-(V4A-g2)
- V4 pad 5: unconnected-(V4A-g1-Pad5) -> Net-(V4A-g1)
- V4 pad 8: unconnected-(V4A-k-Pad8) -> GND-AUD
- V5 pad 1: unconnected-(V5A-g3-Pad1) -> GND-AUD
- V5 pad 4: unconnected-(V5A-g2-Pad4) -> Net-(V5A-g2)
- V5 pad 5: unconnected-(V5A-g1-Pad5) -> Net-(V5A-g1)
- V5 pad 8: unconnected-(V5A-k-Pad8) -> GND-AUD

Commit message: schematic  checked!
Parts:
- added AC-IN1: 1, TestPoint:TestPoint_THTPad_D2.0mm_Drill1.0mm, F.Cu at (456.0, 183.2)
- added AC-IN2: 1, TestPoint:TestPoint_THTPad_D2.0mm_Drill1.0mm, F.Cu at (464.0, 183.2)
- added AC-IN3: 1, TestPoint:TestPoint_THTPad_D2.0mm_Drill1.0mm, F.Cu at (472.0, 183.2)
- added AC-IN4: 1, TestPoint:TestPoint_THTPad_D2.0mm_Drill1.0mm, F.Cu at (521.0, 206.0)
- added AC-IN5: 1, TestPoint:TestPoint_THTPad_D2.0mm_Drill1.0mm, F.Cu at (521.2, 217.0)
- added AC-IN6: 1, TestPoint:TestPoint_THTPad_D2.0mm_Drill1.0mm, F.Cu at (237.2, 73.9)
- added AC-IN7: 1, TestPoint:TestPoint_THTPad_D2.0mm_Drill1.0mm, F.Cu at (241.3, 69.8)
- added AC-IN8: 1, TestPoint:TestPoint_THTPad_D2.0mm_Drill1.0mm, F.Cu at (241.3, 73.9)
- added Audio-A1: 1, TestPoint:TestPoint_THTPad_D3.0mm_Drill1.5mm, F.Cu at (264.8, 24.5)
- added Audio-B1: 1, TestPoint:TestPoint_THTPad_D3.0mm_Drill1.5mm, F.Cu at (264.8, 29.6)
- added BiasA1: 1, TestPoint:TestPoint_Pad_D2.0mm, F.Cu at (269.4, 31.9)
- added BiasB1: 1, TestPoint:TestPoint_Pad_D2.0mm, F.Cu at (269.4, 36.0)
- added C10: 33uF 500V 5R5-ESR, footprints:CAP-TH_BD12.5-P5.00-D0.6-FD, F.Cu at (213.0, 56.4)
- added C11: 18uF 450V ±20%, footprints:CAP-TH_BD10.0-P5.00-D1.0-FD, F.Cu at (225.5, 53.2)
- added C12: 18uF 450V ±20%, footprints:CAP-TH_BD10.0-P5.00-D1.0-FD, F.Cu at (225.5, 64.4)
- added C13: 10uf/100V, footprints:CAP-TH_BD6.3-P2.50-D1.0-FD, F.Cu at (256.5, 51.3)
- added C14: 10uf/100V, footprints:CAP-TH_BD6.3-P2.50-D1.0-FD, F.Cu at (256.5, 58.9)
- added C8: 33uF 500V 5R5-ESR, footprints:CAP-TH_BD12.5-P5.00-D0.6-FD, F.Cu at (398.5, 184.2)
- added C9: 33uF 500V 5R5-ESR, footprints:CAP-TH_BD12.5-P5.00-D0.6-FD, F.Cu at (358.0, 184.0)
- added Choke1: 1, TestPoint:TestPoint_THTPad_D2.0mm_Drill1.0mm, F.Cu at (390.5, 180.2)
- added Choke2: 1, TestPoint:TestPoint_THTPad_D2.0mm_Drill1.0mm, F.Cu at (367.8, 180.0)
- added D1: UF4007_C960666, footprints:DO-41_BD2.4-L4.7-P8.70-D0.9-RD, F.Cu at (446.0, 183.2)
- added D2: UF4007_C960666, footprints:DO-41_BD2.4-L4.7-P8.70-D0.9-RD, F.Cu at (446.0, 190.2)
- added D3: UF4007_C960666, footprints:DO-41_BD2.4-L4.7-P8.70-D0.9-RD, F.Cu at (211.9, 73.4)
- added D4: UF4007_C960666, footprints:DO-41_BD2.4-L4.7-P8.70-D0.9-RD, F.Cu at (268.0, 46.2)
- added D5: UF4007_C960666, footprints:DO-41_BD2.4-L4.7-P8.70-D0.9-RD, F.Cu at (268.0, 50.3)
- added D6: UF4007_C960666, footprints:DO-41_BD2.4-L4.7-P8.70-D0.9-RD, F.Cu at (268.0, 56.3)
- added GND-Mess1: 1, TestPoint:TestPoint_Pad_D2.0mm, F.Cu at (269.4, 40.0)
- added HV-OT1: 1, TestPoint:TestPoint_THTPad_D3.0mm_Drill1.5mm, F.Cu at (382.2, 195.0)
- added HV-OT2: 1, TestPoint:TestPoint_THTPad_D3.0mm_Drill1.5mm, F.Cu at (390.2, 195.0)
- added R24: MOF5WS-47Ω±5%, footprints:RES-TH_BD6.0-L17.5-P21.50-D0.8, F.Cu at (379.0, 186.8)
- added R25: CF3WS-10KΩ±5%_T, footprints:RES-TH_BD5.5-L15.0-P19.00-D0.8, F.Cu at (241.9, 51.0)
- added R26: CF3WS-10KΩ±5%_T, footprints:RES-TH_BD5.5-L15.0-P19.00-D0.8, F.Cu at (241.9, 57.7)
- added R27: CF3WS-10KΩ±5%_T, footprints:RES-TH_BD5.5-L15.0-P19.00-D0.8, F.Cu at (241.9, 64.5)
- added R28: CR1/4W-47K±5%-ST52, footprints:RES-TH_BD2.7-L6.2-P10.20-D0.4, F.Cu at (253.6, 69.8)
- added R29: CR1/4W-15K±5%-OT52, footprints:RES-TH_BD2.7-L6.2-P10.20-D0.4, F.Cu at (253.6, 73.8)
- added R30: MF1/4W-1Ω±1%-ST26, footprints:RES-TH_BD2.7-L6.2-P10.20-D0.4, F.Cu at (273.6, 24.0)
- added R31: MF1/4W-1Ω±1%-ST26, footprints:RES-TH_BD2.7-L6.2-P10.20-D0.4, F.Cu at (273.6, 27.9)
- added R32: CR1/2W-220K±5%-XT52, footprints:RES-TH_BD3.5-L9.0-P13.00-D0.5, F.Cu at (250.4, 43.7)
- added THUMP1: 1, TestPoint:TestPoint_THTPad_D2.0mm_Drill1.0mm, F.Cu at (270.4, 62.4)
- added THUMP2: 1, TestPoint:TestPoint_THTPad_D2.0mm_Drill1.0mm, F.Cu at (270.4, 66.4)
- added U31: 16A 20mm 500V 5mm Plugin Fuse, footprints:FUSE-TH_L22.5-W10.8-P22.50_0031.8201.G, F.Cu at (425.0, 187.2)
- added U32: CR2W-4K7±5%-9T73, footprints:RES-TH_BD5.0-L15.5-P19.50-D0.7, F.Cu at (231.3, 44.4)
- added U33: 3314G-1-503E, footprints:RES-ADJ-SMD_3314G-1-103E, F.Cu at (248.3, 33.4)
- added X1: Switch-ON, TestPoint:TestPoint_THTPad_D2.0mm_Drill1.0mm, F.Cu at (264.3, 62.4)
- added X2: Switch-GND, TestPoint:TestPoint_THTPad_D2.0mm_Drill1.0mm, F.Cu at (264.3, 66.4)
- moved C1 49.8 mm to (502.8, 199.5), turned to 0 degrees
- moved X8 34.9 mm to (549.8, 198.5)
- moved X7 22.2 mm to (542.0, 198.8)
- moved U29 0.78 mm to (136.8, 88.2)
Connections:
- net Net-(U27-Pad2) renamed /Power Amp/Bias-Set
- J2 pad 1: unconnected-(J2-Pad1) -> GND-AUX
- J2 pad 2: unconnected-(J2-Pad2) -> REL-SW
- J2 pad 3: unconnected-(J2-Pad3) -> REL-SW
- J2 pad 4: unconnected-(J2-Pad4) -> Net-(J2-RN)
- J2 pad 5: unconnected-(J2-Pad5) -> Net-(J2-RN)
- J2 pad 6: unconnected-(J2-Pad6) -> GND-AUX
- J3 pad 1: Net-(J3-Pad1) -> GND-AUD
- J4 pad 1: Net-(J3-Pad1) -> GND-AUD
- J4 pad 6: Net-(J3-Pad1) -> GND-AUD
- R5 pad 2: Net-(R5-Pad2) -> GND-AUD
- RELAY1 pad 1: Net-(R5-Pad2) -> Net-(R5-Pad1)
- RELAY1 pad 2: unconnected-(RELAY1-Pad2) -> +12V
- RELAY1 pad 9: unconnected-(RELAY1-Pad9) -> REL-SW
- RELAY2 pad 2: unconnected-(RELAY2-Pad2) -> +12V
- RELAY2 pad 9: unconnected-(RELAY2-Pad9) -> REL-SW
- RELAY3 pad 2: unconnected-(RELAY3-Pad2) -> +12V
- RELAY3 pad 9: unconnected-(RELAY3-Pad9) -> REL-SW
- RV5 pad 1: Net-(Audo-From-FX1-Pad1) -> GND-AUD
- RV5 pad 3: GND-AUD -> Net-(Audo-From-FX1-Pad1)
- RV6 pad 1: Net-(Audo-From-FX1-Pad1) -> GND-AUD
- RV6 pad 3: GND-AUD -> Net-(Audo-From-FX1-Pad1)
- U25 pad 1: HV-C -> Net-(V3A-A/P)
- U3 pad 3: V_Aux_N -> Net-(AC-IN5-Pad1)
- U3 pad 4: V_Aux_P -> Net-(AC-IN4-Pad1)
- V4 pad 1: GND-AUD -> Net-(V4A-g3)
- V4 pad 2: unconnected-(V4B-f-Pad2) -> HEAT1
- V4 pad 3: unconnected-(V4A-a-Pad3) -> Net-(V4A-a)
- V4 pad 7: unconnected-(V4B-f-Pad7) -> HEAT2
- V4 pad 8: GND-AUD -> Net-(V4A-g3)
- V5 pad 1: GND-AUD -> Net-(V5A-g3)
- V5 pad 2: unconnected-(V5B-f-Pad2) -> HEAT1
- V5 pad 3: unconnected-(V5A-a-Pad3) -> Net-(V5A-a)
- V5 pad 7: unconnected-(V5B-f-Pad7) -> HEAT2
- V5 pad 8: GND-AUD -> Net-(V5A-g3)
- X12 pad 1: Net-(J3-Pad1) -> GND-AUD
Routing:
- net HV-A: track 0.00 -> 52.3 mm
- net Net-(D2-A): track 0.00 -> 27.0 mm
- net HV-B: track 0.00 -> 16.5 mm
- net Net-(D1-K): track 0.00 -> 13.7 mm
- net Net-(D1-A): track 0.00 -> 5.65 mm
Other:
- copper layers 6 -> 4
- board text added: "12,6V~"
- board text added: "33uF"
- board text added: "345V~"
- board text added: "GND"

Commit message: updated PCB
Parts:
- removed MH1, MH2: TestPoint, MountingHole:MountingHole_2.2mm_M2_DIN965_Pad_TopBottom
- removed the X1 at (134.4, 186.4)
- removed the X2 at (134.4, 191.5)
- removed X3: 345V - Lila, TestPoint:TestPoint_THTPad_D3.0mm_Drill1.5mm
- removed X4, X6: 3.13V - Grün, TestPoint:TestPoint_THTPad_D3.0mm_Drill1.5mm
- removed X5: CT_HEAT - Schwarz, TestPoint:TestPoint_THTPad_D3.0mm_Drill1.5mm
- removed X7: 12,6V - Rot, TestPoint:TestPoint_THTPad_D3.0mm_Drill1.5mm
- removed X8: 0V - Rot, TestPoint:TestPoint_THTPad_D3.0mm_Drill1.5mm
- added MH3: MountHole, MountingHole:MountingHole_3.5mm_Pad_TopBottom, F.Cu at (123.8, 200.5)
- added MH4: MountHole, MountingHole:MountingHole_3.5mm_Pad_TopBottom, F.Cu at (123.8, 262.5)
- added MH5: MountHole, MountingHole:MountingHole_3.5mm_Pad_TopBottom, F.Cu at (520.5, 269.8)
- added MH6: MountHole, MountingHole:MountingHole_3.5mm_Pad_TopBottom, F.Cu at (520.5, 226.5)
- added MH7: MountHole, MountingHole:MountingHole_3.5mm_Pad_TopBottom, F.Cu at (217.5, 152.0)
- added MH8: MountHole, MountingHole:MountingHole_3.5mm_Pad_TopBottom, F.Cu at (361.5, 152.0)
- added N1: ~, wb50_footprints:NetTie_0.5mm_2Pad, F.Cu at (484.2, 193.2)
- added N2: ~, wb50_footprints:NetTie_0.5mm_2Pad, F.Cu at (377.0, 186.2)
- AC-IN1, AC-IN2, AC-IN3, AC-IN4, AC-IN5, Audio-To-FX1, Audo-From-FX1, THUMP1, THUMP2, X-BS-1, X-BS-2, X-BS-3, X1, X2: footprint TestPoint:TestPoint_THTPad_D2.0mm_Drill1.0mm -> TestPoint:TestPoint_THTPad_D3.0mm_Drill1.5mm
- AC-IN6, AC-IN7, AC-IN8: footprint TestPoint:TestPoint_THTPad_D2.0mm_Drill1.0mm -> TestPoint:TestPoint_THTPad_D4.0mm_Drill2.0mm
- BiasA1, BiasB1, GND-Mess1, U33: moved to B.Cu
- Choke1, Choke2: footprint TestPoint:TestPoint_THTPad_D2.0mm_Drill1.0mm -> TestPoint:TestPoint_THTPad_D2.5mm_Drill1.2mm
- moved U19 471.8 mm to (502.0, 256.0)
- moved U24 352.7 mm to (377.8, 253.8)
- moved R22 342.1 mm to (468.8, 202.5)
- moved U23 336.5 mm to (359.2, 243.2), turned to 180 degrees
- moved U22 330.9 mm to (382.5, 261.8)
- moved R21 325.4 mm to (348.0, 258.8)
- moved D3 323.1 mm to (494.0, 231.0), turned to -90 degrees
- moved U29 317.8 mm to (433.5, 202.0), turned to 180 degrees
- moved U33 315.1 mm to (471.2, 256.0), turned to -90 degrees
- moved U17 304.0 mm to (315.5, 248.8), turned to 180 degrees
- moved C14 302.1 mm to (503.8, 232.5), turned to 180 degrees
- moved U25 301.0 mm to (342.8, 220.2)
- moved C13 300.0 mm to (486.5, 244.0), turned to 180 degrees
- moved U18 295.3 mm to (339.8, 234.0)
- moved R29 295.1 mm to (497.2, 240.2)
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Connections:
- C10 pad 2: GND-PWR -> GND-AUD
- C11 pad 2: GND-PWR -> GND-AUD
- C12 pad 2: GND-PWR -> GND-AUD
- C9 pad 2: GND-PWR -> GND-AUD
Routing:
- net GND-AUD: track 0.00 -> 1016.8 mm
- net +12V: track 0.00 -> 817.0 mm
- net GND-AUX: track 0.00 -> 771.4 mm, vias 0 -> 1
- net /Connectors/NFB_IN: track 0.00 -> 262.8 mm
- net Net-(Audo-From-FX1-Pad1): track 0.00 -> 250.5 mm
- net REL-SW: track 0.00 -> 212.9 mm
- net Net-(RV2-Pad2): track 0.00 -> 210.5 mm
- net Net-(R19-Pad2): track 0.00 -> 205.0 mm, vias 0 -> 1
- net Net-(Audio-To-FX1-Pad1): track 0.00 -> 201.4 mm
- net Net-(RV7-Pad3): track 0.00 -> 161.7 mm
- net Net-(RV4-Pad3): track 0.00 -> 143.5 mm
- net /Power Amp/Bias-Set: track 0.00 -> 143.4 mm
- net Net-(RV3-Pad2): track 0.00 -> 141.4 mm
- net /Phase Inverter/PI_OUT_A: track 0.00 -> 121.8 mm
- net GND-PWR: track 0.00 -> 112.0 mm
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- added copper zone on In2.Cu, net GND-AUD
- added copper zone on In1.Cu, net GND-AUX
- added copper zone on In2.Cu, net GND-PWR
Other:
- board text added: "100k"
- board text added: "10k"
- board text added: "1k"
- board text added: "1k5"
- board text added: "220k"
- board text added: "4k7"
- board text removed: "33uF"
