File: electronics/main/wb50.kicad_pcb (KiCad board)
At the start: 4 copper layers, 405 x 190 mm, 141 parts, among them J1 IN, J2 SW, J3 OUT1, J4 OUT2, U1 XSD366-094, U10 250pF 500V 5%, U11 500pF 500V 5%, U12 500pF 500V 5%, U13 500pF 500V 5%, U14 22n 630V 5%, U15 22n 630V 5%, U16 500pF 500V 5%, U17 22n 630V 5%, U18 470R 500V 2W, U19 100n 630V 5%, U2 L7812CV-DG, U20 CF2WS-82KΩ±5%_T, U21 100pF 500V 5%, U22 CR1/2W-220K±5%-XT52, U23 100n 630V 5%, U24 4n7 630V 5%, U25 22n 630V 5%, U26 22n 630V 5%, U27 CR1/2W-220K±5%-XT52, U28 CR1/2W-220K±5%-XT52, U29 CR-L5W-1KΩJ, U3 AB24S, U30 CR-L5W-1KΩJ, U31 16A 20mm 500V 5mm Plugin Fuse, U32 CR2W-4K7±5%-9T73, U33 3314G-1-503E, U4 CR1/2W-220K±5%-XT52, U5 CR2W-68K±5%-9T73, U6 500pF 500V 5%, U7 4n7 630V 5%, U8 2n2 630V 5%, U9 500pF 500V 5%, X1 Switch-ON, X12 GND_OT, X2 Switch-GND, X9 Audio IN

Commit message: update design
Parts:
- removed X-BS-1: 1, TestPoint:TestPoint_THTPad_D3.0mm_Drill1.5mm
- removed X-BS-2: 2, TestPoint:TestPoint_THTPad_D3.0mm_Drill1.5mm
- removed X-BS-3: 3, TestPoint:TestPoint_THTPad_D3.0mm_Drill1.5mm
- removed X1: Switch-ON, TestPoint:TestPoint_THTPad_D3.0mm_Drill1.5mm
- removed X2: Switch-GND, TestPoint:TestPoint_THTPad_D3.0mm_Drill1.5mm
- added AIR1: VentingHole, MountingHole:MountingHole_4.3mm_M4, F.Cu at (146.2, 198.0)
- added AIR10: VentingHole, MountingHole:MountingHole_4.3mm_M4, F.Cu at (381.0, 227.8)
- added AIR11: VentingHole, MountingHole:MountingHole_4.3mm_M4, F.Cu at (400.2, 242.5)
- added AIR12: VentingHole, MountingHole:MountingHole_4.3mm_M4, F.Cu at (450.2, 211.2)
- added AIR13: VentingHole, MountingHole:MountingHole_4.3mm_M4, F.Cu at (453.8, 240.2)
- added AIR14: VentingHole, MountingHole:MountingHole_4.3mm_M4, F.Cu at (481.8, 238.8)
- added AIR15: VentingHole, MountingHole:MountingHole_4.3mm_M4, F.Cu at (492.2, 183.0)
- added AIR16: VentingHole, MountingHole:MountingHole_4.3mm_M4, F.Cu at (519.0, 195.8)
- added AIR2: VentingHole, MountingHole:MountingHole_4.3mm_M4, F.Cu at (209.2, 264.8)
- added AIR3: VentingHole, MountingHole:MountingHole_4.3mm_M4, F.Cu at (193.2, 207.2)
- added AIR4: VentingHole, MountingHole:MountingHole_4.3mm_M4, F.Cu at (244.2, 208.5)
- added AIR5: VentingHole, MountingHole:MountingHole_4.3mm_M4, F.Cu at (303.8, 207.5)
- added AIR6: VentingHole, MountingHole:MountingHole_4.3mm_M4, F.Cu at (178.2, 246.5)
- added AIR7: VentingHole, MountingHole:MountingHole_4.3mm_M4, F.Cu at (254.0, 242.8)
- added AIR8: VentingHole, MountingHole:MountingHole_4.3mm_M4, F.Cu at (297.8, 224.0)
- added AIR9: VentingHole, MountingHole:MountingHole_4.3mm_M4, F.Cu at (370.2, 232.8)
- added GND-AUD1: 1, TestPoint:TestPoint_THTPad_D3.0mm_Drill1.5mm, F.Cu at (253.5, 152.2)
- added HV-B1: 1, TestPoint:TestPoint_THTPad_D3.0mm_Drill1.5mm, F.Cu at (281.0, 148.2)
- added U34: ST-0-102-C03-N003-RS, footprints:SW-TH_ST-0-102-C03-N003-RS, F.Cu at (199.5, 268.9)
- added U35: MT-0-103-C004-N004-RS, footprints:SW-TH_MT-0-102-C004-N004-RS, F.Cu at (283.0, 263.7)
- moved U9 34.1 mm to (272.0, 254.2)
- moved U10 30.3 mm to (272.0, 260.0)
- moved MH8 18.0 mm to (361.2, 170.0)
- moved U14 17.0 mm to (283.8, 231.5)
- moved R5 10.0 mm to (196.0, 252.2)
- moved R7 6.37 mm to (210.2, 258.0), turned to 0 degrees
- moved U5 5.37 mm to (186.2, 240.5)
- moved MH3 3.00 mm to (123.8, 197.5)
- moved U15 2.80 mm to (295.2, 245.8)
- moved Audio-To-FX1 0.25 mm to (265.8, 152.2)
- moved Audo-From-FX1 0.25 mm to (241.2, 152.2)
Connections:
- MH8 pad 1: unconnected-(MH8-Pad1) -> GND-AUD
- U1 pad 1: Net-(MH1-Pad1) -> unconnected-(U1-Pad1)
- U1 pad 2: Net-(MH2-Pad1) -> unconnected-(U1-Pad2)
Routing:
- net GND-AUD: track 1016.8 -> 1221.7 mm
- net HV-B: track 111.9 -> 234.7 mm
- net Net-(RELAY2-Pad10): track 44.1 -> 59.9 mm
- net GND-AUX: track 771.4 -> 785.1 mm
- net Net-(U35-Pad1): track 18.6 -> 6.95 mm
- net Net-(R15-Pad2): track 33.5 -> 22.3 mm
- net /Connectors/Audio_IN: track 99.8 -> 90.5 mm
- net Net-(RV2-Pad2): track 210.5 -> 217.2 mm
- net Net-(RV7-Pad3): track 161.7 -> 155.6 mm
- net Net-(RV4-Pad3): track 143.5 -> 138.3 mm
- net Net-(R6-Pad1): track 43.5 -> 47.6 mm
- net Net-(R5-Pad1): track 27.6 -> 23.6 mm
- net Net-(J2-RN): track 48.2 -> 46.6 mm
- net REL-SW: track 212.9 -> 214.3 mm
Other:
- board text added: "100nF"
- board text added: "10Meg"
- board text added: "10uF"
- board text added: "15k"
- board text added: "18uF"
- board text added: "1Meg"
- board text added: "1R"
- board text added: "22n"
- board text added: "22uF"
- board text added: "250pF"
- board text added: "2k7"
- board text added: "2n2"
- board text added: "33k"
- board text added: "33uF"
- board text added: "470R"
- board text added: "470k"
- board text added: "47R"
- board text added: "47k"
- board text added: "4n7"
- board text added: "500pF"
- board text added: "68k"
- board text added: "820R"
- board text added: "820nF"
- board text added: "Wechselbalg 50 V1.0 - Christopher Müller 10/25"

Commit message: add fx loop, add new shield
Parts:
- removed Audo-From-FX1: 1, TestPoint:TestPoint_THTPad_D3.0mm_Drill1.5mm
- added AIR17: VentingHole, MountingHole:MountingHole_4.3mm_M4, F.Cu at (251.5, 149.6)
- added AIR18: VentingHole, MountingHole:MountingHole_4.3mm_M4, F.Cu at (293.7, 146.4)
- added AIR19: VentingHole, MountingHole:MountingHole_4.3mm_M4, F.Cu at (272.4, 172.9)
- added AIR20: VentingHole, MountingHole:MountingHole_4.3mm_M4, F.Cu at (520.9, 189.9)
- added AIR21: VentingHole, MountingHole:MountingHole_4.3mm_M4, F.Cu at (492.5, 197.1)
- added AIR22: VentingHole, MountingHole:MountingHole_4.3mm_M4, F.Cu at (516.7, 181.7)
- added Audio-From-FX1: 1, TestPoint:TestPoint_THTPad_D3.0mm_Drill1.5mm, F.Cu at (330.1, 163.1)
- added Audio-From-FX2: 1, TestPoint:TestPoint_THTPad_D3.0mm_Drill1.5mm, F.Cu at (330.0, 157.4)
- added Audio-To-FX2: 1, TestPoint:TestPoint_THTPad_D3.0mm_Drill1.5mm, F.Cu at (337.8, 157.4)
- added C15: 18uF 450V ±20%, footprints:CAP-TH_BD10.0-P5.00-D1.0-FD, F.Cu at (319.1, 167.9)
- added J5: Send, wb50_footprints:WB50_Jack_TRS_6pin_16.2mm, F.Cu at (247.8, 98.1)
- added J6: Return, wb50_footprints:WB50_Jack_TRS_6pin_16.2mm, F.Cu at (275.4, 98.1)
- added R33: 1Meg 500V 250mW, footprints:RES-TH_BD2.4-L6.3-P10.30-D0.6, F.Cu at (319.3, 152.4)
- added R34: CF3WS-10KΩ±5%_T, footprints:RES-TH_BD5.5-L15.0-P19.00-D0.8, F.Cu at (308.1, 163.6)
- added R35: CR1/2WS-470K±5%-ST52, footprints:RES-TH_BD2.7-L6.2-P10.20-D0.4, F.Cu at (348.6, 152.6)
- added R36: CR1/2WS-470K±5%-ST52, footprints:RES-TH_BD2.7-L6.2-P10.20-D0.4, F.Cu at (365.4, 154.4)
- added R37: CF1/4W-1_5KΩ±5%_T52, footprints:RES-TH_BD2.3-L6.5-P10.50-D0.5, F.Cu at (296.3, 161.1)
- added R38: CR1W-10M±5%-6T63, footprints:RES-TH_BD4.5-L11.0-P15.00-D0.7, F.Cu at (236.6, 127.7)
- added R39: CR1/2W-220K±5%-XT52, footprints:RES-TH_BD3.5-L9.0-P13.00-D0.5, F.Cu at (250.5, 113.5)
- added R40: CR1/2W-220K±5%-XT52, footprints:RES-TH_BD3.5-L9.0-P13.00-D0.5, F.Cu at (270.5, 110.2)
- added R41: CF2W-2200Ω±5%_T, footprints:RES-TH_BD5.5-L15.0-P19.00-D0.8, F.Cu at (255.7, 170.1)
- added R42: CR1W-10M±5%-6T63, footprints:RES-TH_BD4.5-L11.0-P15.00-D0.7, F.Cu at (322.0, 132.0)
- added R43: CF2W-2200Ω±5%_T, footprints:RES-TH_BD5.5-L15.0-P19.00-D0.8, F.Cu at (337.4, 169.5)
- added R44: CR1/2W-220K±5%-XT52, footprints:RES-TH_BD3.5-L9.0-P13.00-D0.5, F.Cu at (322.8, 139.2)
- added RV10: Return, wb50_footprints:WB50_Pot_Omeg_PC20BU_P5.00mm, F.Cu at (300.8, 91.2)
- added RV9: Send, wb50_footprints:WB50_Pot_Omeg_PC20BU_P5.00mm, F.Cu at (222.5, 91.2)
- added U36: 47n 630V 5%, wb50_footprints:MUSTARD_CAP_D8.5_L20.5_P25.5, F.Cu at (346.2, 143.2)
- added U37: 470n 630V 5%, wb50_footprints:MUSTARD_CAP_D10_L32_P40.4, F.Cu at (221.2, 120.5)
- added U38: 500pF 500V 5%, wb50_footprints:MICA_CAP_L15.5_W3.6_P8.7, F.Cu at (270.2, 117.0)
- added U39: 220n 630V 5%, wb50_footprints:MUSTARD_CAP_D10_L32_P40.4, F.Cu at (265.8, 129.0)
- added U40: KM1H_4u7_M0405, footprints:CAP-TH_BD4.0-P1.50-D0.5-FD, F.Cu at (263.6, 172.2)
- added U41: 100n 630V 5%, wb50_footprints:MUSTARD_CAP_D10_L32_P40.4, F.Cu at (300.2, 118.8)
- added V6: 12AX7, wb50_footprints:WB50_Socket_Noval_9Pin_D21.0mm_Hole1.8mm, B.Cu at (274.3, 156.5)
- moved GND-AUD1 98.8 mm to (352.1, 159.2)
- moved HV-B1 73.3 mm to (352.0, 166.3)
- moved Audio-To-FX1 73.0 mm to (337.9, 163.1)
- moved X12 57.3 mm to (361.0, 114.7)
- moved X9 32.3 mm to (352.7, 114.7)
- moved J3 20.1 mm to (332.8, 98.0)
- moved J4 20.1 mm to (365.3, 98.0)
- moved AIR16 3.09 mm to (517.8, 198.6)
- moved AC-IN5 2.02 mm to (519.7, 218.3)
- moved AC-IN4 2.00 mm to (519.0, 205.9)
- moved AIR15 1.95 mm to (490.3, 183.1)
Routing:
- net GND-AUD: track 1221.7 -> 1513.5 mm
- net HV-F: track 0.00 -> 126.9 mm
- net Net-(Audio-From-FX1-Pad1): track 250.5 -> 156.2 mm
- net HV-B: track 234.7 -> 141.7 mm
- net GND-AUX: track 785.1 -> 877.7 mm, vias 1 -> 3
- net Net-(V6B-C/K): track 0.00 -> 92.5 mm
- net Net-(Audio-From-FX2-Pad1): track 0.00 -> 83.7 mm
- net Net-(V6A-A/P): track 0.00 -> 76.3 mm
- net Net-(V6B-G): track 0.00 -> 75.8 mm
- net Net-(Audio-To-FX1-Pad1): track 201.4 -> 125.9 mm
- net +12V: track 817.0 -> 886.1 mm
- net Net-(V6A-G): track 0.00 -> 56.8 mm
- net /Connectors/Return: track 0.00 -> 53.1 mm
- net Net-(V6A-C/K): track 0.00 -> 31.2 mm
- net Net-(J5-TN): track 0.00 -> 30.2 mm
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Other:
- outline, holes or cut-outs redrawn
- board text added: "220nF"
- board text added: "2k2"
- board text added: "470nF"
- board text added: "47nF"
- board text added: "6,3V ~"
- board text added: "A1"
- board text added: "B1"
- board text added: "Choke1"
- board text added: "Choke2"
- board text added: "FX-Loop"
- board text added: "GND-AUD"
- board text added: "HV-A"
- board text added: "HV-B"
- board text added: "No-FX-Loop"
- board text added: "Thump1"
- board text added: "Thump2"
