File: electronics/main/wb50.kicad_sch (KiCad schematic)
At the start: 0 parts

Commit message: aux voltage
Other:
- added sheet Aux Power (schematics/auxPower.kicad_sch)
Changed lines of the file:
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@@
+	)
+	(sheet
+		(at 143.51 34.29)
+		(size 39.37 13.97)
+		(exclude_from_sim no)
+		(in_bom yes)
+		(on_board yes)
+		(dnp no)
+		(fields_autoplaced yes)
+		(stroke
+			(width 0.1524)
+			(type solid)
+		)
+		(fill
+			(color 0 0 0 0.0000)
+		)
+		(property "Sheetname" "Aux Power"
+			(at 143.51 33.5784 0)
+			(effects
+				(font
+					(size 1.27 1.27)
+				)
+				(justify left bottom)
+			)
+		)
+		(property "Sheetfile" "schematics/auxPower.kicad_sch"
+			(at 143.51 48.8446 0)
+			(effects
+				(font
+					(size 1.27 1.27)
+				)
+				(justify left top)
+			)
+		)
+		(instances
+			(project "wb50"
+				(path "/6805e3ef-87bd-473d-890f-05ae2da73c1a"
+					(page "7")
+				)
+			)
+		)
 	)
 	(sheet

Commit message: widerstände angelegt
Other:
- sheet Connectors ports: added Audio_IN; removed none
Changed lines of the file:
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@@
 	(paper "A4")
 	(sheet
-		(at 91.44 34.29)
-		(size 36.83 12.7)
+		(at 22.86 80.01)
+		(size 36.83 38.1)
 		(exclude_from_sim no)
 		(in_bom yes)
@@
 		)
 		(property "Sheetname" "Connectors"
-			(at 91.44 33.5784 0)
+			(at 22.86 79.2984 0)
 			(effects
 				(font
@@
 		)
 		(property "Sheetfile" "schematics/connectors.kicad_sch"
-			(at 91.44 47.5746 0)
-			(effects
-				(font
-					(size 1.27 1.27)
-				)
-				(justify left top)
+			(at 22.86 118.6946 0)
+			(effects
+				(font
+					(size 1.27 1.27)
+				)
+				(justify left top)
+			)
+		)
+		(pin "Audio_IN" output
+			(at 59.69 111.76 0)
+			(effects
+				(font
+					(size 1.27 1.27)
+				)
+				(justify right)
 			)
 		)
@@
 	)
 	(sheet
-		(at 44.45 113.03)
-		(size 46.99 12.7)
+		(at 210.82 91.44)
+		(size 46.99 26.67)
 		(exclude_from_sim no)
 		(in_bom yes)
@@
 		)
 		(property "Sheetname" "Power Amp"
-			(at 44.45 112.3184 0)
+			(at 210.82 90.7284 0)
 			(effects
 				(font
@@
 		)
 		(property "Sheetfile" "schematics/powerAmp.kicad_sch"
-			(at 44.45 126.3146 0)
+			(at 210.82 118.6946 0)
 			(effects
 				(font
@@
 	)
 	(sheet
-		(at 110.49 76.2)
-		(size 41.91 13.97)
+		(at 152.4 105.41)
+		(size 19.05 13.97)
 		(exclude_from_sim no)
 		(in_bom yes)
@@
 		)
 		(property "Sheetname" "Phase Inverter"
-			(at 110.49 75.4884 0)
+			(at 152.4 104.6984 0)
 			(effects
 				(font
@@
 		)
 		(property "Sheetfile" "schematics/phaseInverter.kicad_sch"
-			(at 110.49 90.7546 0)
+			(at 152.4 119.9646 0)
 			(effects
 				(font
@@
 	)
 	(sheet
-		(at 40.64 73.66)
-		(size 49.53 15.24)
+		(at 95.25 102.87)
+		(size 21.59 15.24)
 		(exclude_from_sim no)
 		(in_bom yes)
@@
 		)
 		(property "Sheetname" "Pre Amp"
-			(at 40.64 72.9484 0)
+			(at 95.25 102.1584 0)
 			(effects
 				(font
@@
 		)
 		(property "Sheetfile" "schematics/preamp.kicad_sch"
-			(at 40.64 89.4846 0)
+			(at 95.25 118.6946 0)
 			(effects
 				(font
@@
 	)
 	(sheet
-		(at 39.37 34.29)
+		(at 207.01 36.83)
 		(size 40.64 12.7)
 		(exclude_from_sim no)
@@
 		)
 		(property "Sheetname" "Controls"
-			(at 39.37 33.5784 0)
+			(at 207.01 36.1184 0)
 			(effects
 				(font
@@
 		)
 		(property "Sheetfile" "schematics/controls.kicad_sch"
-			(at 39.37 47.5746 0)
+			(at 207.01 50.1146 0)
 			(show_name yes)
 			(effects

Commit message: PI stage ready
Other:
- added sheet Tone Stack (schematics/toneStack.kicad_sch)
- sheet Phase Inverter ports: added NFB_OUT, PI_IN, PI_OUT_A, PI_OUT_B; removed none
- sheet Pre Amp ports: added Audio_IN, PreAmp_OUT; removed none
Changed lines of the file:
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@@
 	(generator_version "9.0")
 	(paper "A4")
+	(wire
+		(pts
+			(xy 144.78 111.76) (xy 170.18 111.76)
+		)
+		(stroke
+			(width 0)
+			(type default)
+		)
+	)
+	(wire
+		(pts
+			(xy 59.69 111.76) (xy 78.74 111.76)
+		)
+		(stroke
+			(width 0)
+			(type default)
+		)
+	)
+	(wire
+		(pts
+			(xy 100.33 107.95) (xy 123.19 107.95)
+		)
+		(stroke
+			(width 0)
+			(type default)
+		)
+	)
 	(sheet
 		(at 22.86 80.01)
@@
 	)
 	(sheet
-		(at 210.82 91.44)
+		(at 223.52 91.44)
 		(size 46.99 26.67)
 		(exclude_from_sim no)
@@
 		)
 		(property "Sheetname" "Power Amp"
-			(at 210.82 90.7284 0)
+			(at 223.52 90.7284 0)
 			(effects
 				(font
@@
 		)
 		(property "Sheetfile" "schematics/powerAmp.kicad_sch"
-			(at 210.82 118.6946 0)
+			(at 223.52 118.6946 0)
 			(effects
 				(font
@@
 	)
 	(sheet
-		(at 152.4 105.41)
+		(at 170.18 104.14)
 		(size 19.05 13.97)
 		(exclude_from_sim no)
@@
 		)
 		(property "Sheetname" "Phase Inverter"
-			(at 152.4 104.6984 0)
+			(at 170.18 103.4284 0)
 			(effects
 				(font
@@
 		)
 		(property "Sheetfile" "schematics/phaseInverter.kicad_sch"
-			(at 152.4 119.9646 0)
-			(effects
-				(font
-					(size 1.27 1.27)
-				)
-				(justify left top)
+			(at 170.18 118.6946 0)
+			(effects
+				(font
+					(size 1.27 1.27)
+				)
+				(justify left top)
+			)
+		)
+		(pin "PI_IN" input
+			(at 170.18 111.76 180)
+			(effects
+				(font
+					(size 1.27 1.27)
+				)
+				(justify left)
+			)
+		)
+		(pin "NFB_OUT" output
+			(at 170.18 107.95 180)
+			(effects
+				(font
+					(size 1.27 1.27)
+				)
+				(justify left)
+			)
+		)
+		(pin "PI_OUT_B" output
+			(at 189.23 113.03 0)
+			(effects
+				(font
+					(size 1.27 1.27)
+				)
+				(justify right)
+			)
+		)
+		(pin "PI_OUT_A" output
+			(at 189.23 110.49 0)
+			(effects
+				(font
+					(size 1.27 1.27)
+				)
+				(justify right)
 			)
 		)
@@
 	)
 	(sheet
-		(at 95.25 102.87)
+		(at 78.74 102.87)
 		(size 21.59 15.24)
 		(exclude_from_sim no)
@@
 		)
 		(property "Sheetname" "Pre Amp"
-			(at 95.25 102.1584 0)
+			(at 78.74 102.1584 0)
 			(effects
 				(font
@@
 		)
 		(property "Sheetfile" "schematics/preamp.kicad_sch"
-			(at 95.25 118.6946 0)
-			(effects
-				(font
-					(size 1.27 1.27)
-				)
-				(justify left top)
+			(at 78.74 118.6946 0)
+			(effects
+				(font
+					(size 1.27 1.27)
+				)
+				(justify left top)
+			)
+		)
+		(pin "Audio_IN" input
+			(at 78.74 111.76 180)
+			(effects
+				(font
+					(size 1.27 1.27)
+				)
+				(justify left)
+			)
+		)
+		(pin "PreAmp_OUT" output
+			(at 100.33 107.95 0)
+			(effects
+				(font
+					(size 1.27 1.27)
+				)
+				(justify right)
 			)
 		)
@@
 				)
 			)
+		)
+	)
+	(sheet
+		(at 123.19 102.87)
+		(size 21.59 15.24)
+		(exclude_from_sim no)
+		(in_bom yes)
+		(on_board yes)
+		(dnp no)
+		(fields_autoplaced yes)
+		(stroke
+			(width 0.1524)
+			(type solid)
+		)
+		(fill
+			(color 0 0 0 0.0000)
+		)
+		(property "Sheetname" "Tone Stack"
+			(at 123.19 102.1584 0)
+			(effects
+				(font
+					(size 1.27 1.27)
+				)
+				(justify left bottom)
+			)
+		)
+		(property "Sheetfile" "schematics/toneStack.kicad_sch"
+			(at 123.19 118.6946 0)
+			(effects
+				(font
+					(size 1.27 1.27)
+				)
+				(justify left top)
+			)
+		)
+		(pin "ToneStack_IN" input
+			(at 123.19 107.95 180)
+			(effects
+				(font
+					(size 1.27 1.27)
+				)
+				(justify left)
+			)
+		)
+		(pin "ToneStack_OUT" output
+			(at 144.78 111.76 0)
+			(effects
+				(font
+					(size 1.27 1.27)
+				)
+				(justify right)
+			)
+		)
+		(instances
+			(project "wb50"
+				(path "/6805e3ef-87bd-473d-890f-05ae2da73c1a"
+					(page "8")
+				)
+			)

Commit message: schematic ready? - check
Other:
- removed sheet Controls
- added sheet Power (schematics/power.kicad_sch)
- sheet Connectors ports: added NFB_IN; removed none
- sheet Power Amp ports: added A_IN, B_IN, Bias-Set; removed none
Changed lines of the file:
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@@
+	(wire
+		(pts
+			(xy 152.4 46.99) (xy 200.66 46.99)
+		)
+		(stroke
+			(width 0)
+			(type default)
+		)
+	)
+	(wire
+		(pts
+			(xy 158.75 107.95) (xy 158.75 88.9)
+		)
+		(stroke
+			(width 0)
+			(type default)
+		)
+	)
+	(wire
+		(pts
+			(xy 158.75 88.9) (xy 59.69 88.9)
+		)
+		(stroke
+			(width 0)
+			(type default)
+		)
+	)
 	(wire
 		(pts
@@
 	(wire
 		(pts
+			(xy 170.18 107.95) (xy 158.75 107.95)
+		)
+		(stroke
+			(width 0)
+			(type default)
+		)
+	)
+	(wire
+		(pts
+			(xy 189.23 110.49) (xy 223.52 110.49)
+		)
+		(stroke
+			(width 0)
+			(type default)
+		)
+	)
+	(wire
+		(pts
+			(xy 189.23 113.03) (xy 223.52 113.03)
+		)
+		(stroke
+			(width 0)
+			(type default)
+		)
+	)
+	(wire
+		(pts
+			(xy 200.66 46.99) (xy 200.66 100.33)
+		)
+		(stroke
+			(width 0)
+			(type default)
+		)
+	)
+	(wire
+		(pts
 			(xy 59.69 111.76) (xy 78.74 111.76)
 		)
@@
 	(wire
 		(pts
+			(xy 200.66 100.33) (xy 223.52 100.33)
+		)
+		(stroke
+			(width 0)
+			(type default)
+		)
+	)
+	(wire
+		(pts
 			(xy 100.33 107.95) (xy 123.19 107.95)
 		)
@@
 			(width 0)
 			(type default)
+		)
+	)
+	(sheet
+		(at 113.03 39.37)
+		(size 39.37 13.97)
+		(exclude_from_sim no)
+		(in_bom yes)
+		(on_board yes)
+		(dnp no)
+		(fields_autoplaced yes)
+		(stroke
+			(width 0.1524)
+			(type solid)
+		)
+		(fill
+			(color 0 0 0 0.0000)
+		)
+		(property "Sheetname" "Power"
+			(at 113.03 38.6584 0)
+			(effects
+				(font
+					(size 1.27 1.27)
+				)
+				(justify left bottom)
+			)
+		)
+		(property "Sheetfile" "schematics/power.kicad_sch"
+			(at 113.03 53.9246 0)
+			(effects
+				(font
+					(size 1.27 1.27)
+				)
+				(justify left top)
+			)
+		)
+		(pin "Bias-Set" output
+			(at 152.4 46.99 0)
+			(effects
+				(font
+					(size 1.27 1.27)
+				)
+				(justify right)
+			)
+		)
+		(instances
+			(project "wb50"
+				(path "/6805e3ef-87bd-473d-890f-05ae2da73c1a"
+					(page "8")
+				)
+			)
 		)
 	)
@@
 			)
 		)
+		(pin "NFB_IN" input
+			(at 59.69 88.9 0)
+			(effects
+				(font
+					(size 1.27 1.27)
+				)
+				(justify right)
+			)
+		)
 		(instances
 			(project "wb50"
@@
 			)
 		)
+		(pin "A_IN" input
+			(at 223.52 110.49 180)
+			(effects
+				(font
+					(size 1.27 1.27)
+				)
+				(justify left)
+			)
+		)
+		(pin "B_IN" input
+			(at 223.52 113.03 180)
+			(effects
+				(font
+					(size 1.27 1.27)
+				)
+				(justify left)
+			)
+		)
+		(pin "Bias-Set" input
+			(at 223.52 100.33 180)
+			(effects
+				(font
+					(size 1.27 1.27)
+				)
+				(justify left)
+			)
+		)
 		(instances
 			(project "wb50"
@@
 	)
 	(sheet
-		(at 143.51 34.29)
+		(at 45.72 39.37)
 		(size 39.37 13.97)
 		(exclude_from_sim no)
@@
 		)
 		(property "Sheetname" "Aux Power"
-			(at 143.51 33.5784 0)
+			(at 45.72 38.6584 0)
 			(effects
 				(font
@@
 		)
 		(property "Sheetfile" "schematics/auxPower.kicad_sch"
-			(at 143.51 48.8446 0)
+			(at 45.72 53.9246 0)
 			(effects
 				(font
@@
 				)
 			)
-		)
-	)
-	(sheet
-		(at 207.01 36.83)
-		(size 40.64 12.7)
-		(exclude_from_sim no)
-		(in_bom yes)
-		(on_board yes)
-		(dnp no)
-		(fields_autoplaced yes)
-		(stroke
-			(width 0.1524)
-			(type solid)
-		)
-		(fill
-			(color 0 0 0 0.0000)
-		)
-		(property "Sheetname" "Controls"
-			(at 207.01 36.1184 0)
-			(effects
-				(font
-					(size 1.27 1.27)
-				)
-				(justify left bottom)
-			)
-		)
-		(property "Sheetfile" "schematics/controls.kicad_sch"
-			(at 207.01 50.1146 0)
-			(show_name yes)
-			(effects
-				(font
-					(size 1.27 1.27)
-				)
-				(justify left top)
-			)
-		)
-		(instances
-			(project "wb50"
-				(path "/6805e3ef-87bd-473d-890f-05ae2da73c1a"
-					(page "2")
-				)
-			)

Commit message: updated PCB
Parts:
- added MH3, MH4, MH5, MH6, MH7, MH8: MountHole, MountingHole:MountingHole_3.5mm_Pad_TopBottom, symbol Connector:TestPoint

Commit message: update design
Parts:
- added AIR1, AIR10, AIR11, AIR12, AIR13, AIR14, AIR15, AIR16, AIR2, AIR3, AIR4, AIR5, AIR6, AIR7, AIR8, AIR9: VentingHole, MountingHole:MountingHole_4.3mm_M4, symbol Connector:TestPoint
Connections:
- net GND-AUD: now reaches MH8.1
- new net GND-AUX: AIR15.1, AIR16.1
Other:
- moved on the sheet: MH3, MH4, MH5, MH6, MH7, MH8

Commit message: add fx loop, add new shield
Parts:
- added AIR17, AIR18, AIR19, AIR20, AIR21, AIR22: VentingHole, MountingHole:MountingHole_4.3mm_M4, symbol Connector:TestPoint
Other:
- sheet Connectors ports: added Return, Send; removed none
- sheet Tone Stack ports: added Return, Send; removed none
